File: kepler-x.kicad_pcb (KiCad board)
At the start: 4 copper layers, 140.5 x 150 mm, 65 parts, among them IC1 SLG46826G, J1 HDMI_C_1.3, J3 Jack_3.5mm_3pin, J4 RasPI_IO_Header_B+, J5 Jack_3.5mm_3pin, J6 Jack_3.5mm_3pin, SW1 SWITCH_INV, SW2 SWITCH_INV, U1 Bus-X68000-ext, U10 74AHC16374, U11 74LVTH162245, U12 TC7MPB9307F, U13 TC7MPB9307F, U14 P0082(DE0-NANO), U15 PLR135-T10, U16 PCM5102, U17 LT1117-3.3, U2 LT1117-3.3, U3 INA3221, U4 74AHC16374, U5 74AHC16374, U6 WM8804GEDS/RV, U7 74AHC16374, U8 74AHC16374, U9 74AHC16374, X1 SG-8002DC(24.576MHz), X2 ASV-xxxMHz, Y1 12MHz

Commit message: Today's version
Parts:
- added D3: Led_Small, LED_SMD:LED_0603_1608Metric_Pad1.05x0.95mm_HandSolder, F.Cu at (142.9, 71.1)
- added D4: Led_Small, LED_SMD:LED_0603_1608Metric_Pad1.05x0.95mm_HandSolder, F.Cu at (205.1, 126.1)
- added D5: Led_Small, LED_SMD:LED_0603_1608Metric_Pad1.05x0.95mm_HandSolder, F.Cu at (210.0, 118.9)
- added D6: D_Schottky_Small, Diode_SMD:D_1206_3216Metric_Pad1.42x1.75mm_HandSolder, B.Cu at (153.0, 91.4)
- added D7: D_Schottky_Small, Diode_SMD:D_1206_3216Metric_Pad1.42x1.75mm_HandSolder, B.Cu at (153.0, 100.3)
- added D8: D_TVS, Diode_SMD:D_1206_3216Metric_Pad1.42x1.75mm_HandSolder, B.Cu at (146.7, 107.3)
- added D9: D_Schottky_Small, Diode_SMD:D_1206_3216Metric_Pad1.42x1.75mm_HandSolder, B.Cu at (146.7, 111.1)
- added J2: Conn_01x02_Male, Connector_PinHeader_2.54mm:PinHeader_1x02_P2.54mm_Vertical, F.Cu at (176.5, 145.2)
- added J7: Conn_01x02_Male, Connector_PinHeader_2.54mm:PinHeader_1x02_P2.54mm_Vertical, F.Cu at (191.0, 145.7)
- added JP4: Jumper_NC_Small, digikey-footprints:PinHeader_1x2_P2.54mm, F.Cu at (72.0, 71.0)
- added JP5: Jumper_NC_Small, Jumper:SolderJumper-2_P1.3mm_Bridged_RoundedPad1.0x1.5mm, F.Cu at (86.0, 96.5)
- added Q1: Q_PNP_BEC, Package_TO_SOT_SMD:SC-59_Handsoldering, B.Cu at (142.9, 91.4)
- added Q2: Q_PNP_BEC, Package_TO_SOT_SMD:SC-59_Handsoldering, B.Cu at (148.6, 91.4)
- added Q3: Q_NPN_BEC, Package_TO_SOT_SMD:SC-59_Handsoldering, B.Cu at (142.9, 101.0)
- added Q4: Q_NPN_BEC, Package_TO_SOT_SMD:SC-59_Handsoldering, B.Cu at (148.6, 101.0)
- added Q5: Q_NPN_BEC, Package_TO_SOT_SMD:SC-59_Handsoldering, B.Cu at (141.6, 107.3)
- added Q6: Q_NPN_BEC, Package_TO_SOT_SMD:SC-59_Handsoldering, B.Cu at (138.4, 114.9)
- added R10: R_Small_US, Resistor_SMD:R_0603_1608Metric_Pad0.98x0.95mm_HandSolder, B.Cu at (139.7, 92.1)
- added R11: R_Small_US, Resistor_SMD:R_0603_1608Metric_Pad0.98x0.95mm_HandSolder, B.Cu at (139.7, 100.3)
- added R12: R_Small_US, Resistor_SMD:R_0603_1608Metric_Pad0.98x0.95mm_HandSolder, B.Cu at (146.4, 95.2)
- added R13: R_Small_US, Resistor_SMD:R_0603_1608Metric_Pad0.98x0.95mm_HandSolder, B.Cu at (146.4, 97.2)
- added R14: R_Small_US, Resistor_SMD:R_0603_1608Metric_Pad0.98x0.95mm_HandSolder, B.Cu at (142.2, 111.1)
- added R15: R_Small_US, Resistor_SMD:R_0603_1608Metric_Pad0.98x0.95mm_HandSolder, B.Cu at (141.6, 104.8)
- added R6: 1K, Resistor_SMD:R_0603_1608Metric_Pad0.98x0.95mm_HandSolder, F.Cu at (121.1, 125.5)
- added R7: 1K, Resistor_SMD:R_0603_1608Metric_Pad0.98x0.95mm_HandSolder, F.Cu at (214.3, 118.9)
- added R8: 10K, Resistor_SMD:R_0603_1608Metric_Pad0.98x0.95mm_HandSolder, F.Cu at (134.0, 89.1)
- added R9: 1K, Resistor_SMD:R_0603_1608Metric_Pad0.98x0.95mm_HandSolder, F.Cu at (116.7, 125.5)
- added RP7: R_PACK4, Resistor_SMD:R_Array_Convex_4x0603, F.Cu at (44.0, 45.0)
- added U18: TLP785, Package_DIP:DIP-4_W7.62mm, F.Cu at (136.5, 109.9)
- D1, D2: footprint Diode_SMD:D_MELF_Handsoldering -> Diode_SMD:D_1206_3216Metric_Pad1.42x1.75mm_HandSolder
- J3, J5, J6: value Jack_3.5mm_3pin -> AudioJack3
- moved JP2 55.9 mm to (79.7, 103.0)
- moved J5 50.2 mm to (164.5, 47.6)
- moved J3 49.3 mm to (164.5, 97.8)
- moved U6 5.72 mm to (146.7, 76.8)
- moved C4 5.14 mm to (149.2, 89.5)
- moved C5 5.08 mm to (144.1, 89.5)
- moved Y1 5.08 mm to (149.1, 85.1)
Connections:
- J3 pad R: (no net) -> Net-(D7-Pad2)
- J3 pad S: (no net) -> GND
- J3 pad T: (no net) -> Net-(D6-Pad1)
- J5 pad R: (no net) -> Net-(J5-PadR)
- J5 pad S: (no net) -> GNDA
- J5 pad T: (no net) -> Net-(J5-PadT)
- J6 pad R: (no net) -> Net-(D8-Pad1)
- J6 pad S: (no net) -> unconnected-(J6-PadS)
- J6 pad T: (no net) -> Net-(D8-Pad2)
- JP1 pad 2: /i2C_SCL -> /I2C_SCL
- JP2 pad 2: /i2C_SCL -> /I2C_SCL
- U1 pad B48: (no net) -> /ExBGACK
- U14 pad JP1_7: /I2C_SCK -> /I2C_SCL
- U16 pad 10: unconnected-(U16-Pad10) -> GND
- U16 pad 11: unconnected-(U16-Pad11) -> GND
- U16 pad 16: unconnected-(U16-Pad16) -> GND
- U16 pad 6: Net-(J3-Pad2) -> Net-(J5-PadT)
- U16 pad 7: Net-(J3-Pad3) -> Net-(J5-PadR)
- U3 pad 10: unconnected-(U3-Pad10) -> Net-(RP7-Pad4)
- U3 pad 13: unconnected-(U3-Pad13) -> Net-(RP7-Pad1)
- U3 pad 16: unconnected-(U3-Pad16) -> +3V3
- U3 pad 4: VCC -> +3V3
- U3 pad 5: unconnected-(U3-Pad5) -> Net-(JP4-Pad1)
- U3 pad 6: unconnected-(U3-Pad6) -> /I2C_SCL
- U3 pad 7: unconnected-(U3-Pad7) -> /I2C_SDA
- U3 pad 8: unconnected-(U3-Pad8) -> Net-(RP7-Pad2)
- U3 pad 9: unconnected-(U3-Pad9) -> Net-(RP7-Pad3)
- U6 pad 1: unconnected-(U6-Pad1) -> /I2C_SCL
- U6 pad 2: unconnected-(U6-Pad2) -> Net-(D3-Pad2)
- U6 pad 3: unconnected-(U6-Pad3) -> /I2C_SDA
- U6 pad 4: unconnected-(U6-Pad4) -> Net-(D5-Pad2)
- U6 pad 5: unconnected-(U6-Pad5) -> Net-(D4-Pad2)
- U6 pad 6: unconnected-(U6-Pad6) -> /iEXRESET
- U9 pad 1: unconnected-(U9-Pad1) -> /iB_AO_OE
- X2 pad 3: /iCLK24M576 -> Net-(JP5-Pad2)
Routing:
- net /MIDI_OUT: track 0.00 -> 76.0 mm
- net /MIDI_IN: track 0.00 -> 75.6 mm
- net Net-(D8-Pad2): track 0.00 -> 27.8 mm
- net Net-(D8-Pad1): track 0.00 -> 22.9 mm
- net Net-(D6-Pad1): track 0.00 -> 18.9 mm
- net Net-(R12-Pad2): track 0.00 -> 14.4 mm
- net Net-(R10-Pad1): track 0.00 -> 13.4 mm, vias 0 -> 2
- net GND: track 64.5 -> 76.8 mm, vias 2 -> 7
- net Net-(R13-Pad1): track 0.00 -> 11.8 mm
- net (no net): track 0.00 -> 8.12 mm
- net VCC: track 2.28 -> 8.67 mm
- net Net-(R15-Pad1): track 0.00 -> 4.81 mm
- net Net-(R11-Pad2): track 0.00 -> 4.27 mm
- net Net-(C4-Pad1): track 0.00 -> 3.62 mm
- net Net-(D7-Pad2): track 0.00 -> 3.56 mm
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- added copper zone on In1.Cu, net +3V3
- added copper zone on In2.Cu, net GND

Commit message: DRC free version
Parts:
- removed JP2: Jumper_NC_Small, digikey-footprints:PinHeader_1x2_P2.54mm
- removed JP5: Jumper_NC_Small, Jumper:SolderJumper-2_P1.3mm_Bridged_RoundedPad1.0x1.5mm
- removed TP1: TestPoint, TestPoint:TestPoint_THTPad_2.0x2.0mm_Drill1.0mm
- removed X1: SG-8002DC(24.576MHz), Oscillator:Oscillator_SeikoEpson_SG-8002DC
- C10, C3, C6, D2, D3, D4, D5, JP3, R6, R7, R8, R9, RP1, RP2, RP3, RP4, RP7, TP4: moved to B.Cu
- J4: footprint Module:Raspberry_Pi_Zero_Socketed_THT_FaceDown_MountingHoles -> x68000-ext:Raspberry_Pi_Zero_Socketed_THT_FaceDown_MountingHoles
- JP4: footprint digikey-footprints:PinHeader_1x2_P2.54mm -> Jumper:SolderJumper-2_P1.3mm_Bridged_RoundedPad1.0x1.5mm; moved to B.Cu
- U10: value 74AHC16374 -> 74LVTH162245; footprint Housings_SSOP:SSOP-48_7.5x15.9mm_Pitch0.635mm -> x68000-ext:SSOP-48_7.5x15.9mm_Pitch0.635mm; moved to F.Cu
- U11: value 74LVTH162245 -> WM8804GEDS/RV; footprint Housings_SSOP:SSOP-48_7.5x15.9mm_Pitch0.635mm -> x68000-ext:WM8804GEDS&slash_RV
- U17, U2: footprint Package_TO_SOT_SMD:TO-263-3_TabPin2 -> Package_TO_SOT_SMD:SOT-223-3_TabPin2
- U4, U5, U8, U9: footprint Housings_SSOP:SSOP-48_7.5x15.9mm_Pitch0.635mm -> x68000-ext:SSOP-48_7.5x15.9mm_Pitch0.635mm
- U6: value WM8804GEDS/RV -> 74AHC16374; footprint x68000-ext:WM8804GEDS&slash_RV -> x68000-ext:SSOP-48_7.5x15.9mm_Pitch0.635mm
- U7: footprint Housings_SSOP:SSOP-48_7.5x15.9mm_Pitch0.635mm -> x68000-ext:SSOP-48_7.5x15.9mm_Pitch0.635mm; moved to B.Cu
- moved J7 169.0 mm to (59.7, 39.4)
- moved J2 163.4 mm to (52.1, 39.4)
- moved JP1 134.9 mm to (64.8, 108.6), turned to -90 degrees
- moved U6 123.4 mm to (59.8, 164.5)
- moved TP4 114.9 mm to (67.3, 66.0), turned to 180 degrees
- moved R7 93.0 mm to (121.9, 108.6)
- moved D5 92.7 mm to (118.1, 106.7), turned to 180 degrees
- moved D4 88.8 mm to (118.1, 108.6), turned to 180 degrees
- moved JP3 86.9 mm to (142.9, 49.5)
- moved C10 80.1 mm to (137.8, 52.7), turned to 180 degrees
- moved U11 75.3 mm to (121.9, 96.5)
- moved C3 64.0 mm to (121.3, 101.6), turned to 180 degrees
- moved TP2 60.2 mm to (158.1, 66.7)
- moved TP3 59.0 mm to (154.3, 66.7)
- moved C6 55.6 mm to (129.5, 99.1), turned to 90 degrees
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Connections:
- net Net-(R2-Pad1) renamed /+12V_S
- net Net-(R3-Pad1) renamed /VCC2_S
- net Net-(R3-Pad2) renamed /VCC2
- IC1 pad 13: Net-(IC1-Pad13) -> /I2C_SCL
- J2 pad 1: Net-(J2-Pad1) -> /VCC_S
- J7 pad 1: Net-(J2-Pad1) -> /VCC_S
- JP1 pad 1: Net-(IC1-Pad13) -> Net-(IC1-Pad12)
- JP1 pad 2: /I2C_SCL -> /I2C_SDA
- R1 pad 1: Net-(J2-Pad1) -> /VCC_S
- U1 pad A49: Net-(J2-Pad1) -> /VCC_S
- U1 pad A50: Net-(J2-Pad1) -> /VCC_S
- U1 pad B49: VCC -> /VCC_S
- U1 pad B50: VCC -> /VCC_S
- U10 pad 1: /iB_DO_OE -> GND
- U10 pad 11: /ExDB6 -> unconnected-(U10-Pad11)
- U10 pad 12: /ExDB7 -> unconnected-(U10-Pad12)
- U10 pad 13: /ExDB8 -> /ExBG
- U10 pad 14: /ExDB9 -> Net-(SW2-Pad2)
- U10 pad 16: /ExDB10 -> /ExEXRESET
- U10 pad 17: /ExDB11 -> /ExEXACK
- U10 pad 18: (no net) -> +3V3
- U10 pad 19: /ExDB12 -> /ExDTC
- U10 pad 2: /ExDB0 -> unconnected-(U10-Pad2)
- U10 pad 20: /ExDB13 -> /ExVSYNC
- U10 pad 22: /ExDB14 -> /ExHSYNC
- U10 pad 23: /ExDB15 -> /ExCLK10M
- U10 pad 24: /iB_DO_OE -> GND
- U10 pad 25: /iB_DO_CK -> GND
- U10 pad 26: /iSB15 -> /iCLK10M
- U10 pad 27: /iSB14 -> /iHSYNC
- U10 pad 29: /iSB13 -> /iVSYNC
- U10 pad 3: /ExDB1 -> unconnected-(U10-Pad3)
- U10 pad 30: /iSB12 -> /iDTC
- U10 pad 31: (no net) -> +3V3
- U10 pad 32: /iSB11 -> /iEXACK
- U10 pad 33: /iSB10 -> /iEXRESET
- U10 pad 35: /iSB9 -> /iIACK
- U10 pad 36: /iSB8 -> /iBG
- U10 pad 37: /iSB7 -> unconnected-(U10-Pad37)
- U10 pad 38: /iSB6 -> unconnected-(U10-Pad38)
- U10 pad 40: /iSB5 -> unconnected-(U10-Pad40)
- U10 pad 41: /iSB4 -> unconnected-(U10-Pad41)
- U10 pad 43: /iSB3 -> unconnected-(U10-Pad43)
- U10 pad 44: /iSB2 -> unconnected-(U10-Pad44)
- U10 pad 46: /iSB1 -> unconnected-(U10-Pad46)
- U10 pad 47: /iSB0 -> unconnected-(U10-Pad47)
- U10 pad 48: /iB_DO_CK -> GND
- U10 pad 5: /ExDB2 -> unconnected-(U10-Pad5)
- U10 pad 6: /ExDB3 -> unconnected-(U10-Pad6)
- U10 pad 8: /ExDB4 -> unconnected-(U10-Pad8)
- U10 pad 9: /ExDB5 -> unconnected-(U10-Pad9)
- U11 pad 1: GND -> /I2C_SCL
- U11 pad 10: GND -> Net-(C4-Pad1)
- U11 pad 11: unconnected-(U11-Pad11) -> Net-(C5-Pad1)
- U11 pad 12: unconnected-(U11-Pad12) -> /I2S_DATA_IN
- U11 pad 13: /ExBG -> /I2S_DATA
- U11 pad 14: Net-(SW2-Pad2) -> /I2S_BCLK
- U11 pad 15: GND -> /I2S_LRCK
- U11 pad 16: /ExEXRESET -> /I2S_MCLK
- U11 pad 17: /ExEXACK -> Net-(TR1-Pad1)
- U11 pad 18: (no net) -> GND
- U11 pad 19: /ExDTC -> +3V3
- U11 pad 2: unconnected-(U11-Pad2) -> Net-(D3-Pad2)
- U11 pad 20: /ExHSYNC -> Net-(U11-Pad20)
- U11 pad 3: unconnected-(U11-Pad3) -> /I2C_SDA
- U11 pad 4: GND -> Net-(D5-Pad2)
- U11 pad 5: unconnected-(U11-Pad5) -> Net-(D4-Pad2)
- U11 pad 6: unconnected-(U11-Pad6) -> /iEXRESET
- U11 pad 8: unconnected-(U11-Pad8) -> GND
- U14 pad JP1_17: /BUS_MODE3 -> /I2S_DATA
- U14 pad JP1_18: /BUS_MODE2 -> /BUS_MODE0
- U14 pad JP1_19: /BUS_MODE1 -> /I2S_LRCK
- U14 pad JP1_20: /BUS_MODE0 -> /BUS_MODE1
- U14 pad JP1_21: /I2S_MCLK -> /I2S_BCLK
- U14 pad JP1_22: /I2S_DATA -> /BUS_MODE2
- U14 pad JP1_23: /I2S_LRCK -> /I2S_MCLK
- U14 pad JP1_24: /I2S_BCLK -> /BUS_MODE3
- U14 pad JP1_36: /iPCL -> /iEXPCL
- U14 pad JP2_11: Net-(D2-Pad1) -> unconnected-(U14-PadJP2_11)
- U15 pad 3: Net-(U15-Pad3) -> Net-(U11-Pad20)
- U3 pad 10: Net-(RP7-Pad4) -> Net-(RP7-Pad2)
- U3 pad 12: Net-(J2-Pad1) -> /VCC_S
- U3 pad 8: Net-(RP7-Pad2) -> Net-(RP7-Pad4)
- U4 pad 18: (no net) -> +3V3
- U4 pad 31: (no net) -> +3V3
- U5 pad 18: (no net) -> +3V3
- U5 pad 31: (no net) -> +3V3
- U6 pad 1: /I2C_SCL -> /iB_DI_OE
- U6 pad 10: Net-(C4-Pad1) -> GND
- U6 pad 11: Net-(C5-Pad1) -> /iSB6
- U6 pad 12: /I2S_DATA_IN -> /iSB7
- U6 pad 13: /I2S_DATA -> /iSB8
- U6 pad 14: /I2S_BCLK -> /iSB9
- U6 pad 15: /I2S_LRCK -> GND
- U6 pad 16: /I2S_MCLK -> /iSB10
- U6 pad 17: Net-(TR1-Pad1) -> /iSB11
- U6 pad 18: GND -> +3V3
- U6 pad 19: +3V3 -> /iSB12
- U6 pad 2: Net-(D3-Pad2) -> /iSB0
- U6 pad 20: Net-(U15-Pad3) -> /iSB13
- U6 pad 3: /I2C_SDA -> /iSB1
- U6 pad 4: Net-(D5-Pad2) -> GND
- U6 pad 5: Net-(D4-Pad2) -> /iSB2
- U6 pad 6: /iEXRESET -> /iSB3
- U6 pad 8: GND -> /iSB4
- U6 pad 9: unconnected-(U6-Pad9) -> /iSB5
- U7 pad 1: /iB_DI_OE -> /iB_AO_OE
- U7 pad 11: /iSB6 -> /ExAB22
- U7 pad 12: /iSB7 -> /ExAB23
- U7 pad 13: /iSB8 -> /ExFC0
- U7 pad 14: /iSB9 -> /ExFC1
- U7 pad 16: /iSB10 -> /ExFC2
- U7 pad 17: /iSB11 -> unconnected-(U7-Pad17)
- U7 pad 18: (no net) -> +3V3
- U7 pad 19: /iSB12 -> unconnected-(U7-Pad19)
- U7 pad 2: /iSB0 -> /ExAB16
- U7 pad 20: /iSB13 -> unconnected-(U7-Pad20)
- U7 pad 22: /iSB14 -> unconnected-(U7-Pad22)
- U7 pad 23: /iSB15 -> unconnected-(U7-Pad23)
- U7 pad 24: /iB_DI_OE -> /iB_AO_OE
- U7 pad 25: /iB_DI_CK -> /iB_AO_CK_U
- U7 pad 26: /ExDB15 -> /iSB15
- U7 pad 27: /ExDB14 -> /iSB14
- U7 pad 29: /ExDB13 -> /iSB13
- U7 pad 3: /iSB1 -> /ExAB17
- U7 pad 30: /ExDB12 -> /iSB12
- U7 pad 31: (no net) -> +3V3
- U7 pad 32: /ExDB11 -> /iSB11
- U7 pad 33: /ExDB10 -> /iSB10
- U7 pad 35: /ExDB9 -> /iSB9
- U7 pad 36: /ExDB8 -> /iSB8
- U7 pad 37: /ExDB7 -> /iSB7
- U7 pad 38: /ExDB6 -> /iSB6
- U7 pad 40: /ExDB5 -> /iSB5
- U7 pad 41: /ExDB4 -> /iSB4
- U7 pad 43: /ExDB3 -> /iSB3
- U7 pad 44: /ExDB2 -> /iSB2
- U7 pad 46: /ExDB1 -> /iSB1
- U7 pad 47: /ExDB0 -> /iSB0
- U7 pad 48: /iB_DI_CK -> /iB_AO_CK_U
- U7 pad 5: /iSB2 -> /ExAB18
- U7 pad 6: /iSB3 -> /ExAB19
- U7 pad 8: /iSB4 -> /ExAB20
- U7 pad 9: /iSB5 -> /ExAB21
- U8 pad 11: /ExAB22 -> /ExAB6
- U8 pad 12: /ExAB23 -> /ExAB7
- U8 pad 13: /ExFC0 -> /ExAB8
- U8 pad 14: /ExFC1 -> /ExAB9
- U8 pad 16: /ExFC2 -> /ExAB10
- U8 pad 17: unconnected-(U8-Pad17) -> /ExAB11
- U8 pad 18: (no net) -> +3V3
- U8 pad 19: unconnected-(U8-Pad19) -> /ExAB12
- U8 pad 2: /ExAB16 -> unconnected-(U8-Pad2)
- U8 pad 20: unconnected-(U8-Pad20) -> /ExAB13
- U8 pad 22: unconnected-(U8-Pad22) -> /ExAB14
- U8 pad 23: unconnected-(U8-Pad23) -> /ExAB15
- U8 pad 25: /iB_AO_CK_U -> /iB_AO_CK_L
- U8 pad 3: /ExAB17 -> /ExAB1
- U8 pad 31: (no net) -> +3V3
- U8 pad 48: /iB_AO_CK_U -> /iB_AO_CK_L
- U8 pad 5: /ExAB18 -> /ExAB2
- U8 pad 6: /ExAB19 -> /ExAB3
- U8 pad 8: /ExAB20 -> /ExAB4
- U8 pad 9: /ExAB21 -> /ExAB5
- U9 pad 1: /iB_AO_OE -> /iB_DO_OE
- U9 pad 11: /ExAB6 -> /ExDB6
- U9 pad 12: /ExAB7 -> /ExDB7
- U9 pad 13: /ExAB8 -> /ExDB8
- U9 pad 14: /ExAB9 -> /ExDB9
- U9 pad 16: /ExAB10 -> /ExDB10
- U9 pad 17: /ExAB11 -> /ExDB11
- U9 pad 18: (no net) -> +3V3
- U9 pad 19: /ExAB12 -> /ExDB12
- U9 pad 2: unconnected-(U9-Pad2) -> /ExDB0
- U9 pad 20: /ExAB13 -> /ExDB13
- U9 pad 22: /ExAB14 -> /ExDB14
- U9 pad 23: /ExAB15 -> /ExDB15
- U9 pad 24: /iB_AO_OE -> /iB_DO_OE
- U9 pad 25: /iB_AO_CK_L -> /iB_DO_CK
- U9 pad 3: /ExAB1 -> /ExDB1
- U9 pad 31: (no net) -> +3V3
- U9 pad 48: /iB_AO_CK_L -> /iB_DO_CK
- U9 pad 5: /ExAB2 -> /ExDB2
- U9 pad 6: /ExAB3 -> /ExDB3
- U9 pad 8: /ExAB4 -> /ExDB4
- U9 pad 9: /ExAB5 -> /ExDB5
- X2 pad 3: Net-(JP5-Pad2) -> /iCLK24M576
Routing:
- net VCC: track 8.67 -> 397.4 mm, vias 0 -> 8
- net /I2C_SCL: track 0.00 -> 260.0 mm, vias 0 -> 8
- net /I2C_SDA: track 0.00 -> 244.9 mm, vias 0 -> 6
- net /I2S_BCLK: track 0.00 -> 209.1 mm, vias 0 -> 6
- net /iSB1: track 0.00 -> 185.4 mm, vias 0 -> 11
- net /iSB3: track 0.00 -> 182.7 mm, vias 0 -> 11
- net /iSB0: track 0.00 -> 182.7 mm, vias 0 -> 8
- net /iSB2: track 0.00 -> 179.6 mm, vias 0 -> 8
- net /iSB5: track 0.00 -> 179.0 mm, vias 0 -> 11
- net /iSB4: track 0.00 -> 178.2 mm, vias 0 -> 8
- net /iSB7: track 0.00 -> 178.0 mm, vias 0 -> 11
- net /iSB9: track 0.00 -> 175.6 mm, vias 0 -> 11
- net /iSB8: track 0.00 -> 175.2 mm, vias 0 -> 8
- net /iSB13: track 0.00 -> 174.7 mm, vias 0 -> 11
- net /I2S_DATA: track 0.00 -> 174.4 mm, vias 0 -> 4
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- added copper zone on In1.Cu, net +3.3VA
- added copper zone on B.Cu, net /VCC_S
- added copper zone on F.Cu, net /VCC_S
- added copper zone on In2.Cu, net GNDA

Commit message: Alpha version
Parts:
- added J8: Conn_02x07_Odd_Even, Connector_PinHeader_2.54mm:PinHeader_2x08_P2.54mm_Vertical, F.Cu at (103.5, 89.5)
- added J9: Conn_01x02_Male, Connector_PinHeader_2.54mm:PinHeader_1x02_P2.54mm_Vertical, F.Cu at (84.5, 170.8)
- added JP2: Jumper_NO_Small, Jumper:SolderJumper-2_P1.3mm_Open_RoundedPad1.0x1.5mm, B.Cu at (92.1, 157.5)
- added JP5: Jumper_NO_Small, Jumper:SolderJumper-2_P1.3mm_Open_RoundedPad1.0x1.5mm, B.Cu at (94.6, 157.5)
- J3: value AudioJack3 -> MIDI OUT
- J6: value AudioJack3 -> MIDI IN
- moved R7 43.2 mm to (142.2, 70.5), turned to 90 degrees
- moved D4 41.9 mm to (142.2, 74.3), turned to -90 degrees
- moved R9 40.6 mm to (140.3, 70.5), turned to 90 degrees
- moved D5 39.3 mm to (140.3, 74.3), turned to -90 degrees
- moved R6 38.1 mm to (138.4, 70.5), turned to 90 degrees
- moved D3 36.6 mm to (138.4, 74.3), turned to -90 degrees
- moved C3 32.8 mm to (144.1, 78.1), turned to 0 degrees
- moved U11 29.8 mm to (148.6, 83.2)
- moved C6 28.8 mm to (154.3, 84.5)
- moved C5 22.8 mm to (151.1, 72.4), turned to 180 degrees
- moved R8 18.1 mm to (121.9, 92.7), turned to 180 degrees
- moved C4 16.8 mm to (146.7, 72.4)
- moved Y1 16.6 mm to (146.7, 76.2), turned to 0 degrees
- moved JP1 12.7 mm to (52.1, 108.6)
- moved J2 8.03 mm to (59.7, 41.9), turned to 180 degrees
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Connections:
- J4 pad 10: unconnected-(J4-Pad10) -> Net-(J4-Pad10)
- J4 pad 2: VCC -> Net-(J4-Pad2)
- J4 pad 26: unconnected-(J4-Pad26) -> /FM_CLK4M
- J4 pad 27: unconnected-(J4-Pad27) -> /FM_RD
- J4 pad 28: unconnected-(J4-Pad28) -> /FM_WR
- J4 pad 29: unconnected-(J4-Pad29) -> /FM_IRQ
- J4 pad 31: unconnected-(J4-Pad31) -> /FM_PHY
- J4 pad 32: unconnected-(J4-Pad32) -> /FM_DAT
- J4 pad 33: unconnected-(J4-Pad33) -> /FM_LRCK
- J4 pad 36: unconnected-(J4-Pad36) -> /FM_SCLK
- J4 pad 37: unconnected-(J4-Pad37) -> /FM_SDATA
- J4 pad 4: VCC -> Net-(J4-Pad2)
- J4 pad 40: unconnected-(J4-Pad40) -> /iEXRESET
- J4 pad 8: unconnected-(J4-Pad8) -> Net-(J4-Pad8)
- U14 pad JP2_31: /FMWR -> /FM_WR
- U3 pad 17: (no net) -> GND
Routing:
- net /FM_IRQ: track 0.00 -> 143.8 mm, vias 0 -> 2
- net /FM_SCLK: track 0.00 -> 142.5 mm, vias 0 -> 2
- net /FM_DAT: track 0.00 -> 141.9 mm, vias 0 -> 2
- net /FM_SDATA: track 0.00 -> 140.1 mm, vias 0 -> 3
- net /FM_RD: track 0.00 -> 137.9 mm, vias 0 -> 3
- net /FM_WR: track 0.00 -> 136.8 mm, vias 0 -> 3
- net /FM_PHY: track 0.00 -> 136.5 mm, vias 0 -> 3
- net /FM_CLK4M: track 0.00 -> 136.1 mm
- net /FM_LRCK: track 0.00 -> 135.3 mm, vias 0 -> 3
- net /iEXRESET: track 128.4 -> 243.5 mm, vias 2 -> 5
- net /MIDI_OUT: track 78.5 -> 172.1 mm, vias 0 -> 2
- net /MIDI_IN: track 80.0 -> 159.7 mm, vias 0 -> 1
- net VCC: track 397.4 -> 447.2 mm
- net /I2C_SDA: track 244.9 -> 293.8 mm, vias 6 -> 10
- net /I2C_SCL: track 260.0 -> 305.1 mm, vias 8 -> 10
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Other:
- board text added: "+"
- board text added: "+5V IN"
- board text added: "DVI"
- board text added: "G"
- board text added: "S/PDIF IN"
- board text added: "S/PDIF OUT"

Commit message: current version (DE0 Nano is upside down :-( )
Parts:
- added C13: 0.1uF, Capacitor_SMD:C_0603_1608Metric_Pad1.08x0.95mm_HandSolder, F.Cu at (52.3, 104.1)
- added C14: 0.1uF, Capacitor_SMD:C_0603_1608Metric_Pad1.08x0.95mm_HandSolder, F.Cu at (65.0, 153.7)
- added C15: 0.1uF, Capacitor_SMD:C_0603_1608Metric_Pad1.08x0.95mm_HandSolder, F.Cu at (65.0, 173.5)
- added C16: 0.1uF, Capacitor_SMD:C_0603_1608Metric_Pad1.08x0.95mm_HandSolder, F.Cu at (65.0, 134.1)
- added C17: 0.1uF, Capacitor_SMD:C_0603_1608Metric_Pad1.08x0.95mm_HandSolder, F.Cu at (56.6, 85.1)
- added C18: 0.1uF, Capacitor_SMD:C_0603_1608Metric_Pad1.08x0.95mm_HandSolder, F.Cu at (55.4, 74.4)
- added C19: 2.2nF, Capacitor_SMD:C_0603_1608Metric_Pad1.08x0.95mm_HandSolder, B.Cu at (155.6, 52.1)
- added C20: 2.2nF, Capacitor_SMD:C_0603_1608Metric_Pad1.08x0.95mm_HandSolder, B.Cu at (155.6, 54.0)
- added G***: LOGO, x68000-ext:Kepler-chan-40x40, B.Cu at (122.7, 125.0)
- added R16: 10K, Resistor_SMD:R_0603_1608Metric_Pad0.98x0.95mm_HandSolder, B.Cu at (151.8, 52.1)
- added R17: 10K, Resistor_SMD:R_0603_1608Metric_Pad0.98x0.95mm_HandSolder, B.Cu at (151.8, 54.0)
- moved C2 2.65 mm to (57.1, 57.7)
- moved J2 2.54 mm to (59.7, 44.5)
- moved J7 2.54 mm to (52.1, 44.5)
- moved C1 2.29 mm to (57.1, 48.3)
- moved C12 1.42 mm to (142.9, 45.1)
- moved C11 1.27 mm to (142.9, 41.2)
- moved C10 1.27 mm to (137.8, 54.0)
- moved C7 1.27 mm to (137.8, 52.1)
- moved C8 1.27 mm to (142.9, 61.0)
- moved C9 1.27 mm to (148.6, 54.0)
- moved U16 1.27 mm to (143.5, 55.9)
- moved JP3 1.27 mm to (142.9, 50.8)
Connections:
- U16 pad 6: Net-(J5-PadT) -> Net-(U16-Pad6)
- U16 pad 7: Net-(J5-PadR) -> Net-(U16-Pad7)
Routing:
- net GND: track 192.1 -> 206.9 mm, vias 78 -> 84
- net Net-(J5-PadR): track 16.8 -> 8.16 mm
- net +3V3: track 120.0 -> 128.3 mm, vias 40 -> 44
- net Net-(U16-Pad6): track 0.00 -> 7.68 mm
- net Net-(J5-PadT): track 29.1 -> 21.5 mm
- net Net-(U16-Pad7): track 0.00 -> 6.42 mm
- net VCC: track 447.2 -> 441.6 mm
- net /VCC_S: track 57.1 -> 54.6 mm
- net GNDA: track 4.16 -> 6.24 mm, vias 2 -> 4
- net /I2S_DATA: track 192.3 -> 190.5 mm
- net /I2S_LRCK: track 191.9 -> 190.1 mm
- net +3.3VA: track 18.9 -> 17.9 mm
- net /I2C_SCL: track 305.1 -> 304.6 mm
- removed copper zone on F.Cu, net /VCC_S
Other:
- board text added: "Developed by @kunichiko. September 2022"
- board text added: "Kepler-X"
- board text added: "Multifunction expansion board for X680x0 series"
- board text added: "壱號機 V1.0.0"
