File: kepler-x.kicad_pcb (KiCad board)
At the start: 4 copper layers, 140.5 x 150 mm, 105 parts, among them IC1 SLG46826G, J1 HDMI_C_1.3, J2 Conn_01x02_Male, J3 MIDI OUT, J4 RasPI_IO_Header_B+, J5 AudioJack3, J6 MIDI IN, J7 Conn_01x02_Male, J8 Conn_02x07_Odd_Even, J9 Conn_01x02_Male, Q1 Q_PNP_BEC, Q2 Q_PNP_BEC, Q3 Q_NPN_BEC, Q4 Q_NPN_BEC, Q5 Q_NPN_BEC, Q6 Q_NPN_BEC, SW1 SWITCH_INV, SW2 SWITCH_INV, U1 Bus-X68000-ext, U10 74LVTH162245, U11 WM8804GEDS/RV, U12 TC7MPB9307F, U13 TC7MPB9307F, U14 P0082(DE0-NANO), U15 PLR135-T10, U16 PCM5102, U17 LT1117-3.3, U18 TLP785, U2 LT1117-3.3, U3 INA3221, U4 74AHC16374, U5 74AHC16374, U6 74AHC16374, U7 74AHC16374, U8 74AHC16374, U9 74AHC16374, X2 ASV-xxxMHz, Y1 12MHz

Commit message: Fix upside down foot print.
Parts:
- added R18: 10K, Resistor_SMD:R_0603_1608Metric_Pad0.98x0.95mm_HandSolder, B.Cu at (121.9, 94.6)
- U14: footprint x68000-ext:MODULE_P0082_BOTTOMMOUNT -> x68000-ext:MODULE_P0082_TOPMOUNT
- U18: value TLP785 -> H11L1; footprint Package_DIP:DIP-4_W7.62mm -> Package_DIP:DIP-6_W7.62mm
- moved D2 22.9 mm to (85.7, 74.9)
- moved U18 1.27 mm to (135.2, 109.2)
Connections:
- U14 pad JP1_11: Net-(D2-Pad1) -> unconnected-(U14-PadJP1_11)
- U14 pad JP2_11: unconnected-(U14-PadJP2_11) -> Net-(D2-Pad1)
- U18 pad 3: /MIDI_IN -> unconnected-(U18-Pad3)
- U18 pad 4: +3V3 -> /MIDI_IN
Routing:
- net /iHSYNC: track 85.0 -> 37.1 mm, vias 4 -> 1
- net /iBG: track 84.3 -> 36.5 mm, vias 4 -> 1
- net /iVSYNC: track 81.5 -> 33.7 mm, vias 4 -> 1
- net /iEXACK: track 84.3 -> 36.5 mm, vias 4 -> 1
- net /iSB7: track 178.0 -> 130.8 mm, vias 11 -> 8
- net /FM_SCLK: track 142.5 -> 95.7 mm
- net /FM_DAT: track 141.9 -> 95.1 mm
- net /FM_RD: track 137.9 -> 91.1 mm, vias 3 -> 2
- net /iSB9: track 175.6 -> 128.8 mm, vias 11 -> 8
- net /iSB5: track 179.0 -> 132.2 mm, vias 11 -> 8
- net /iSB11: track 172.6 -> 125.8 mm, vias 11 -> 8
- net /BUS_MODE2: track 62.0 -> 108.8 mm, vias 2 -> 4
- net /BUS_MODE0: track 65.0 -> 111.8 mm, vias 2 -> 4
- net /iSB13: track 174.7 -> 127.9 mm, vias 11 -> 8
- net /iSB3: track 182.7 -> 135.9 mm, vias 11 -> 8
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Other:
- board text added: "I2C SCL Pull-up"
- board text added: "I2C SDA Pull-up"
- board text added: "Terrasic DE0 Nano"
