File: kepler-x.kicad_sch (KiCad schematic)
At the start: 20 parts, among them U1 Bus-X68000-ext, U6 WM8804GEDS{slash}RV

Commit message: Today's version
Parts:
- added C1, C11: 10uF, Capacitor_THT:CP_Radial_D5.0mm_P2.50mm, symbol Device:C_Polarized_Small_US
- added C10, C6, C7: 0.1uF, Capacitor_SMD:C_0603_1608Metric, symbol Device:C_Small
- added C12, C2: 100uF, Capacitor_THT:CP_Radial_D5.0mm_P2.50mm, symbol Device:C_Polarized_Small_US
- added C3: 1uF, Capacitor_THT:CP_Radial_D5.0mm_P2.50mm, symbol Device:C_Small
- added C4: 15pF, Capacitor_THT:CP_Radial_D5.0mm_P2.50mm, symbol Device:C_Small
- added C5: 15pF, Capacitor_SMD:C_0603_1608Metric_Pad1.08x0.95mm_HandSolder, symbol Device:C_Small
- added C8, C9: 2.2uF, Capacitor_SMD:C_0603_1608Metric, symbol Device:C_Small
- added D1, D2: D_Schottky_Small, Diode_SMD:D_MELF_Handsoldering, symbol device:D_Schottky_Small
- added IC1: SLG46826G, x68000-ext:SOP65P640X120-20N, symbol x68000-ext:SLG46826G
- added J1: HDMI_C_1.3, digikey-footprints:HDMI_Mini_Female_2001-1-2-21-00-BK, symbol Connector:HDMI_C_1.3
- added J2: HDMI_A, Connector_HDMI:HDMI_A_Kycon_KDMIX-SL1-NS-WS-B15_VerticalRightAngle, symbol Connector:HDMI_A
- added J3: Jack_3.5mm_3pin, Connector_Audio:Jack_3.5mm_CUI_SJ-3523-SMT_Horizontal, symbol w_connectors:Jack_3.5mm_3pin
- added J4: RasPI_IO_Header_B+, symbol w_connectors:RasPI_IO_Header_B+
- added JP1, JP2, JP3: Jumper_NC_Small, symbol device:Jumper_NC_Small
- added R1, R2, R3: R_Shunt_US, symbol Device:R_Shunt_US
- added R4, R5: R_US, symbol Device:R_US
- added RP5, RP6: 270, symbol device:R_PACK4
- added TP1, TP2, TP3, TP4: TestPoint, symbol Connector:TestPoint
- added U15: PLR135-T10, PLR135-T10_PLT133-T10W, symbol x68000-ext:PLR135-T10
- added U16: PCM5102, Package_SO:TSSOP-20_4.4x6.5mm_P0.65mm, symbol Audio:PCM5102
- added U17, U2: LT1117-3.3, symbol Regulator_Linear:LT1117-3.3
- added U3: INA3221, Housings_DFN_QFN:QFN-16-1EP_4x4mm_Pitch0.65mm, symbol x68000-ext:INA3221
- added X1: SG-8002DC(24.576MHz), Oscillator:Oscillator_SeikoEpson_SG-8002DC, symbol Oscillator:SG-8002DC
- added X2: ASV-xxxMHz, Oscillator:Oscillator_SMD_Abracon_ASV-4Pin_7.0x5.1mm, symbol Oscillator:ASV-xxxMHz
- added Y1: 12MHz, symbol Device:Crystal_Small
- U14: renamed from U?; footprint MODULE_P0082_BOTTOMMOUNT -> x68000-ext:MODULE_P0082_BOTTOMMOUNT
- gave numbers to parts that had none: 15
Connections:
- net IBOUTDB_OE is gone; now on net iRW: U14.JP1_31 (GPIO_024)
- net iBOUTDB_CLK is gone; now on net iIDDIR: U14.JP1_32 (GPIO_025)
- net +12V: now also R2.4; no longer U1.A22 (+12V), U1.A23 (+12V)
- net +3V3: now also U6.19 (DVDD), U6.7 (PVDD), C2.1, C3.1, C6.1, C7.1, IC1.20 (VDD), IC1.7 (VDD2), U16.1 (CPVDD), U16.20 (DVDD), U2.2 (VO), X1.8 (Vcc), X2.4 (Vdd); no longer U14.JP1_29 (GPIO-0_VCC3P3)
- net ExEXPWON: now also U12.13 (B6)
- net ExIACK2: now also SW2.1
- net ExIACK4: now also SW2.3
- net ExIRQ2: now also SW1.1
- net ExIRQ4: now also SW1.3
- net GND: now also TR1.3 (GND), U14.JP2_12 (GPIO-1_GND), U14.JP2_30 (GPIO-1_GND), U14.S1 (SHIELD), U14.S2 (SHIELD), U14.S3 (SHIELD), U14.S4 (SHIELD), U6.18 (DGND), U6.8 (PGND), C1.2, C10.2, C11.2, C12.2, C2.2, C3.2, C4.2, C5.2, C6.2, C7.2, C8.2, IC1.10 (GND), J1.1 (D2S), J1.10 (CKS), J1.13 (GND), J1.4 (D1S), J1.7 (D0S), J1.SH, J2.11 (CKS), J2.17 (GND), J2.2 (D2S), J2.5 (D1S), J2.8 (D0S), J2.SH, J4.14 (GND), J4.17 (3V3), J4.20 (GND), J4.25 (GND), J4.30 (GND), J4.34 (GND), J4.39 (GND), J4.6 (GND), J4.9 (GND), JP3.1, U15.2 (GND), U16.19 (DGND), U16.3 (CPGND), U17.1 (GND), U2.1 (GND), U3.3 (GND), X1.4 (GND), X2.2 (GND)
- net VCC: now also TR1.2 (VCC), C1.1, C11.1, D1.2 (A), D2.2 (A), J4.2 (5V), J4.4 (5V), R1.4, U15.1 (VCC), U17.3 (VI), U2.3 (VI), U3.4 (VS); no longer U1.A49 (VCC1), U1.A50 (VCC1), U14.JP1_11 (GPIO-0_VCC_SYS)
- net iAS: now also U14.JP1_26 (GPIO_021), IC1.15 (IO4)
- net iBG: now also U14.JP2_8 (GPIO_15)
- net iBGACK: now also U14.JP1_40 (GPIO_033)
- net iBR: now also U14.JP1_39 (GPIO_032)
- net iCLK10M: now also U14.JP2_1 (GPIO_1_IN0)
- net iDONE: now also U14.JP1_33 (GPIO_026)
- net iDTACK: now also U14.JP1_34 (GPIO_027)
- net iDTC: now also U14.JP2_5 (GPIO_12)
- net iEXACK: now also U14.JP2_6 (GPIO_13)
- net iEXOWN: now also U14.JP1_37 (GPIO_030)
- net iEXREQ: now also U14.JP1_35 (GPIO_028)
- net iEXRESET: now also U14.JP2_38 (GPIO_131)
- net iHSYNC: now also U14.JP2_4 (GPIO_11)
- net iIACK: now also U14.JP2_7 (GPIO_14)
- net iIRQ: now also U14.JP1_38 (GPIO_031)
- net iLDS: now also U14.JP1_27 (GPIO_022)
- net iSB0: now also U14.JP2_9 (GPIO_16); no longer U14.JP1_18 (GPIO_013)
- net iSB1: now also U14.JP2_10 (GPIO_17); no longer U14.JP1_17 (GPIO_012)
- net iSB10: now also U14.JP2_21 (GPIO_116); no longer U14.JP1_6 (GPIO_03)
- net iSB11: now also U14.JP2_22 (GPIO_117); no longer U14.JP1_5 (GPIO_02)
- net iSB12: now also U14.JP2_23 (GPIO_118); no longer U14.JP1_4 (GPIO_01)
- net iSB13: now also U14.JP2_24 (GPIO_119); no longer U14.JP1_3 (GPIO_0_IN1)
- net iSB14: now also U14.JP2_25 (GPIO_120); no longer U14.JP1_2 (GPIO_00)
- net iSB15: now also U14.JP2_26 (GPIO_121); no longer U14.JP1_1 (GPIO_0_IN0)
- net iSB2: now also U14.JP2_13 (GPIO_18); no longer U14.JP1_16 (GPIO_011)
- net iSB3: now also U14.JP2_14 (GPIO_19); no longer U14.JP1_15 (GPIO_010)
- net iSB4: now also U14.JP2_15 (GPIO_110); no longer U14.JP1_14 (GPIO_09)
- net iSB5: now also U14.JP2_16 (GPIO_111); no longer U14.JP1_13 (GPIO_08)
- net iSB6: now also U14.JP2_17 (GPIO_112); no longer U14.JP1_10 (GPIO_07)
- net iSB7: now also U14.JP2_18 (GPIO_113); no longer U14.JP1_9 (GPIO_06)
- net iSB8: now also U14.JP2_19 (GPIO_114); no longer U14.JP1_8 (GPIO_05)
- net iSB9: now also U14.JP2_20 (GPIO_115); no longer U14.JP1_7 (GPIO_04)
- net iUDS: now also U14.JP1_28 (GPIO_023)
- net iVSYNC: now also U14.JP2_2 (GPIO_10)
- net iEXPWON: now reaches RP1.3 (P3), U12.7 (A6)
- net iEXPWON: now also J4.7 (GPIO4/GPCLK0)
- net at U1.A42 (VCC2): now also U1.A43 (VCC2), R3.1
- net at U6.10 (XOP): now also C4.1, Y1.1
- net at U6.11 (XIN): now also C5.1, Y1.2
- net I2S_DATA_IN: now reaches U6.12 (DOUT)
- net I2S_DATA_IN: now also U14.JP1_25 (GPIO_020)
- net I2S_DATA: now reaches U6.13 (DIN)
- net I2S_DATA: now also U14.JP1_22 (GPIO_017), J4.38 (GPIO20), U16.14 (DIN)
- net I2S_BCLK: now reaches U6.14 (BCLK)
- net I2S_BCLK: now also U14.JP1_24 (GPIO_019), J4.12 (GPIO18/PCM_CLK/CE0-1/PWM0/GPIO_GEN1), U16.13 (BCK)
- net I2S_LRCK: now reaches U6.15 (LRCLK)
- net I2S_LRCK: now also U14.JP1_23 (GPIO_018), J4.35 (GPIO19), U16.15 (LRCK)
- net I2S_MCLK: now reaches U6.16 (MCLK)
- net I2S_MCLK: now also U14.JP1_21 (GPIO_016), U16.12 (SCK)
- net at U6.17 (TX0): now also TR1.1 (VIN)
- net at U6.20 (RX0): now also U15.3 (VOUT)
- net iPCL: now reaches U14.JP1_36 (GPIO_029)
- net at U14.JP2_11 (GPIO-1_VCC_SYS): now also U14.JP1_11 (GPIO-0_VCC_SYS), D2.1 (K)
- net FM_CLK4M: now reaches U14.JP2_27 (GPIO_122)
- net FM_RD: now reaches U14.JP2_28 (GPIO_123)
- net iCLK24M576: now reaches U14.JP2_3 (GPIO_1_IN1)
- net iCLK24M576: now also X1.5 (OUT), X2.3 (OUT)
- net FMWR: now reaches U14.JP2_31 (GPIO_124)
- net FM_IRQ: now reaches U14.JP2_32 (GPIO_125)
- net FM_PHY: now reaches U14.JP2_33 (GPIO_126)
- net FM_DAT: now reaches U14.JP2_34 (GPIO_127)
- net FM_LRCK: now reaches U14.JP2_35 (GPIO_128)
- net FM_SCLK: now reaches U14.JP2_36 (GPIO_129)
- net FM_SDATA: now reaches U14.JP2_37 (GPIO_130)
- net MIDI_IN: now reaches U14.JP2_39 (GPIO_132)
- net MIDI_OUT: now reaches U14.JP2_40 (GPIO_133)
- net IBOUTDB_CLK renamed iB_DO_CK
- net iB_DO_CK: now also IC1.11 (IO6)
- net iBINAL_CLK renamed iB_AI_CK
- net iB_AI_CK: now also U4.25 (2CLK), U4.48 (1CLK), IC1.1 (IO14); no longer U14.JP1_22 (GPIO_017)
- net iBINAL_OE renamed iB_AI_OE_L
- net iB_AI_OE_L: now also IC1.3 (IO12); no longer U14.JP1_21 (GPIO_016)
- removed net iBINAU_CLK: U14.JP1_20 (GPIO_015), U4.25 (2CLK), U4.48 (1CLK)
- net iBINAU_OE renamed iB_AI_OE_U
- net iB_AI_OE_U: now also IC1.2 (IO13); no longer U14.JP1_19 (GPIO_014)
- net iBINDB_CLK renamed iB_DI_CK
- net iB_DI_CK: now also IC1.8 (IO8); no longer U14.JP1_24 (GPIO_019)
- net iBINDB_OE renamed iB_DI_OE
- net iB_DI_OE: now also IC1.9 (IO7); no longer U14.JP1_23 (GPIO_018)
- net iBOUTAL_CLK renamed iB_AO_CK_L
- net iB_AO_CK_L: now also IC1.5 (IO10); no longer U14.JP1_28 (GPIO_023)
- net iBOUTAL_OE renamed iB_AO_OE
- net iB_AO_OE: now also U8.1 (1~{OE}), U8.24 (2~{OE}), IC1.6 (IO9); no longer U14.JP1_27 (GPIO_022)
- net iBOUTAU_CLK renamed iB_AO_CK_U
- net iB_AO_CK_U: now also IC1.4 (IO11); no longer U14.JP1_26 (GPIO_021)
- removed net iBOUTAU_OE: U14.JP1_25 (GPIO_020), U8.1 (1~{OE}), U8.24 (2~{OE})
- net iBOUTDB_OE renamed iB_DO_OE
- net iB_DO_OE: now also IC1.14 (IO5)
- new net: R2.1, U1.A22 (+12V), U1.A23 (+12V)
- new net: R1.1, U1.A49 (VCC1), U1.A50 (VCC1)
- new net: TP4.1, X1.1 (OE), X2.1 (EN)
- new net: R2.2, U3.15 (IN+2)
- new net: R2.3, U3.14 (IN-2)
- new net: C10.1, U16.18 (LDOO)
- new net: D1.1 (K), J1.18 (+5V), J2.18 (+5V), R4.1, R5.1
- new net: J1.16 (SDA), J2.16 (SDA), R5.2, TP2.1
- new net: R1.2, U3.12 (IN+1)
- new net: R1.3, U3.11 (IN-1)
- new net: IC1.12 (SDA), JP2.1
- new net: J1.6 (D1-), J2.6 (D1-), RP5.5 (R4)
- new net: J1.5 (D1+), J2.4 (D1+), RP5.6 (R3)
- new net: J1.3 (D2-), J2.3 (D2-), RP5.7 (R2)
- new net: J1.2 (D2+), J2.1 (D2+), RP5.8 (R1)
- new net: J1.15 (SCL), J2.15 (SCL), R4.2, TP3.1
- new net: J3.2 (T), U16.6 (OUTL)
- new net: J3.3 (R), U16.7 (OUTR)
- new net: C9.1, U16.2 (CAPP)
- new net: C9.2, U16.4 (CAPM)
- new net: C8.1, U16.5 (VNEG)
- new net: R3.3, U3.1 (IN-3)
- new net: R3.2, U3.2 (IN+3)
- new net: IC1.13 (SCL), JP1.1
- new net: R3.4, TP1.1
- new net: J1.11 (CK+), J2.10 (CK+), RP6.6 (R3)
- new net: J1.12 (CK-), J2.12 (CK-), RP6.5 (R4)
- new net: J1.8 (D0+), J2.7 (D0+), RP6.8 (R1)
- new net: J1.9 (D0-), J2.9 (D0-), RP6.7 (R2)
- new net +3.3VA: C12.1, U16.8 (AVDD), U17.2 (VO)
- new net BUS_MODE0: IC1.16 (IO3), U14.JP1_20 (GPIO_015)
- new net BUS_MODE1: IC1.17 (IO2), U14.JP1_19 (GPIO_014)
- new net BUS_MODE2: IC1.18 (IO1), U14.JP1_18 (GPIO_013)
- new net BUS_MODE3: IC1.19 (IO0), U14.JP1_17 (GPIO_012)
- new net GNDA: J3.1 (S), JP3.2, U16.9 (AGND)
- new net HDMI_CLKn: RP6.4 (P4), U14.JP1_16 (GPIO_011)
- new net HDMI_CLKp: RP6.3 (P3), U14.JP1_15 (GPIO_010)
- new net HDMI_D0n: RP6.2 (P2), U14.JP1_13 (GPIO_08)
- new net HDMI_D0p: RP6.1 (P1), U14.JP1_10 (GPIO_07)
- new net HDMI_D1n: RP5.4 (P4), U14.JP1_9 (GPIO_06)
- new net HDMI_D1p: RP5.3 (P3), U14.JP1_8 (GPIO_05)
- new net HDMI_D2n: RP5.2 (P2), U14.JP1_5 (GPIO_02)
- new net HDMI_D2p: RP5.1 (P1), U14.JP1_6 (GPIO_03)
- new net I2C_SCK: U14.JP1_7 (GPIO_04)
- new net I2C_SCL: J4.5 (GPIO1-R1/GPIO3-R2/SCL0/SCL1)
- new net I2C_SDA: J4.3 (GPIO0-R1/GPIO2-R2/SDA0/SDA1), U14.JP1_14 (GPIO_09)
- new net RasPi_SPI_CS0: J4.24 (GPIO8/CE0-N), U14.JP1_3 (GPIO_0_IN1)
- new net RasPi_SPI_MISO: J4.21 (GPIO9/SPI_MISO0), U14.JP1_4 (GPIO_01)
- new net RasPi_SPI_MOSI: J4.19 (GPIO10/SPI_MOSI0), U14.JP1_2 (GPIO_00)
- new net RasPi_SPI_SCLK: J4.23 (GPIO11/SPI_SCKL0), U14.JP1_1 (GPIO_0_IN0)
- new net i2C_SCL: JP1.2, JP2.2
- no-connect marks 33 -> 57
Other:
- note added: "Alternative"
- moved on the sheet: TR1, U1, U14A, U14B, U6

Commit message: Add fooprints
Parts:
- removed R1, R2, R3: R_Shunt_US, symbol Device:R_Shunt_US
- added R1, R2, R3: R100 (0.1Ω), Resistor_SMD:R_2512_6332Metric_Pad1.40x3.35mm_HandSolder, symbol Device:R_Small_US
- J4: footprint (none) -> Module:Raspberry_Pi_Zero_Socketed_THT_FaceDown_MountingHoles
- JP1, JP2: footprint (none) -> digikey-footprints:PinHeader_1x2_P2.54mm
- JP3: footprint (none) -> Jumper:SolderJumper-2_P1.3mm_Bridged_RoundedPad1.0x1.5mm
- R4, R5: footprint (none) -> Resistor_SMD:R_0603_1608Metric_Pad0.98x0.95mm_HandSolder
- RP1, RP2, RP3, RP4, RP5, RP6: footprint (none) -> Resistor_SMD:R_Array_Convex_4x0603
- SW1, SW2: footprint (none) -> Pin_Headers:Pin_Header_Straight_1x03
- TP1, TP2, TP3, TP4: footprint (none) -> TestPoint:TestPoint_THTPad_2.0x2.0mm_Drill1.0mm
- U15: footprint PLR135-T10_PLT133-T10W -> x68000-ext:XDCR_PLT133_T10W
- U17, U2: footprint (none) -> Package_TO_SOT_SMD:TO-263-3_TabPin2
- Y1: footprint (none) -> Crystal:Crystal_HC49-U_Vertical
Connections:
- net +12V: now also U3.14 (IN-2), R2.2
- net VCC: now also U3.11 (IN-1), R1.2
- net at U1.A22 (+12V), U1.A23 (+12V): now also U3.15 (IN+2), R2.1
- net at U1.A42 (VCC2), U1.A43 (VCC2): now also U3.2 (IN+3), R3.1
- net at U1.A49 (VCC1), U1.A50 (VCC1): now also U3.12 (IN+1), R1.1
- net at U3.1 (IN-3): now also TP1.1, R3.2

Commit message: Today's version
Parts:
- removed J2: HDMI_A, Connector_HDMI:HDMI_A_Kycon_KDMIX-SL1-NS-WS-B15_VerticalRightAngle, symbol Connector:HDMI_A
- added H1, H2: MountingHole, MountingHole:MountingHole_3.7mm, symbol Mechanical:MountingHole
- added H3, H4: MountingHole, MountingHole:MountingHole_2.7mm_M2.5, symbol Mechanical:MountingHole
- added J2: USB_B_Micro, symbol Connector:USB_B_Micro
- added J5, J6: Jack_3.5mm_3pin, Connector_Audio:Jack_3.5mm_Switronic_ST-005-G_horizontal, symbol w_connectors:Jack_3.5mm_3pin
- C10, C6, C7, C8, C9: footprint Capacitor_SMD:C_0603_1608Metric -> Capacitor_SMD:C_0603_1608Metric_Pad1.08x0.95mm_HandSolder
- C3, C4: footprint Capacitor_THT:CP_Radial_D5.0mm_P2.50mm -> Capacitor_SMD:C_0603_1608Metric_Pad1.08x0.95mm_HandSolder
- J3: footprint Connector_Audio:Jack_3.5mm_CUI_SJ-3523-SMT_Horizontal -> Connector_Audio:Jack_3.5mm_Switronic_ST-005-G_horizontal
Connections:
- net ExAB1: now also U9.3 (1Q2); no longer U9.22 (2Q7)
- net ExAB10: now also U9.16 (2Q3); no longer U9.9 (1Q6)
- net ExAB11: now also U9.17 (2Q4); no longer U9.8 (1Q5)
- net ExAB12: now also U9.19 (2Q5); no longer U9.6 (1Q4)
- net ExAB13: now also U9.20 (2Q6); no longer U9.5 (1Q3)
- net ExAB14: now also U9.22 (2Q7); no longer U9.3 (1Q2)
- net ExAB15: now also U9.23 (2Q8); no longer U9.2 (1Q1)
- net ExAB16: now also U8.2 (1Q1); no longer U8.23 (2Q8)
- net ExAB17: now also U8.3 (1Q2); no longer U8.22 (2Q7)
- net ExAB18: now also U8.5 (1Q3); no longer U8.20 (2Q6)
- net ExAB19: now also U8.6 (1Q4); no longer U8.19 (2Q5)
- net ExAB2: now also U9.5 (1Q3); no longer U9.20 (2Q6)
- net ExAB20: now also U8.8 (1Q5); no longer U8.17 (2Q4)
- net ExAB21: now also U8.9 (1Q6); no longer U8.16 (2Q3)
- net ExAB22: now also U8.11 (1Q7); no longer U8.14 (2Q2)
- net ExAB23: now also U8.12 (1Q8); no longer U8.13 (2Q1)
- net ExAB3: now also U9.6 (1Q4); no longer U9.19 (2Q5)
- net ExAB4: now also U9.8 (1Q5); no longer U9.17 (2Q4)
- net ExAB5: now also U9.9 (1Q6); no longer U9.16 (2Q3)
- net ExAB6: now also U9.11 (1Q7); no longer U9.14 (2Q2)
- net ExAB7: now also U9.12 (1Q8); no longer U9.13 (2Q1)
- net ExAB8: now also U9.13 (2Q1); no longer U9.12 (1Q8)
- net ExAB9: now also U9.14 (2Q2); no longer U9.11 (1Q7)
- net ExDB0: now also U10.2 (1Q1); no longer U10.23 (2Q8)
- net ExDB1: now also U10.3 (1Q2); no longer U10.22 (2Q7)
- net ExDB10: now also U10.16 (2Q3); no longer U10.9 (1Q6)
- net ExDB11: now also U10.17 (2Q4); no longer U10.8 (1Q5)
- net ExDB12: now also U10.19 (2Q5); no longer U10.6 (1Q4)
- net ExDB13: now also U10.20 (2Q6); no longer U10.5 (1Q3)
- net ExDB14: now also U10.22 (2Q7); no longer U10.3 (1Q2)
- net ExDB15: now also U10.23 (2Q8); no longer U10.2 (1Q1)
- net ExDB2: now also U10.5 (1Q3); no longer U10.20 (2Q6)
- net ExDB3: now also U10.6 (1Q4); no longer U10.19 (2Q5)
- net ExDB4: now also U10.8 (1Q5); no longer U10.17 (2Q4)
- net ExDB5: now also U10.9 (1Q6); no longer U10.16 (2Q3)
- net ExDB6: now also U10.11 (1Q7); no longer U10.14 (2Q2)
- net ExDB7: now also U10.12 (1Q8); no longer U10.13 (2Q1)
- net ExDB8: now also U10.13 (2Q1); no longer U10.12 (1Q8)
- net ExDB9: now also U10.14 (2Q2); no longer U10.11 (1Q7)
- net ExFC0: now also U8.13 (2Q1); no longer U8.12 (1Q8)
- net ExFC1: now also U8.14 (2Q2); no longer U8.11 (1Q7)
- net ExFC2: now also U8.16 (2Q3); no longer U8.9 (1Q6)
- net GND: now also J2.5 (GND), J2.6 (Shield)
- net iB_AO_OE: no longer U9.1 (1~{OE})
- net iSB0: now also U10.47 (1D1), U8.47 (1D1), U9.47 (1D1); no longer U10.26 (2D8), U8.26 (2D8), U9.26 (2D8)
- net iSB1: now also U10.46 (1D2), U8.46 (1D2), U9.46 (1D2); no longer U10.27 (2D7), U8.27 (2D7), U9.27 (2D7)
- net iSB10: now also U10.33 (2D3), U8.33 (2D3), U9.33 (2D3); no longer U10.40 (1D6), U8.40 (1D6), U9.40 (1D6)
- net iSB11: now also U10.32 (2D4), U8.32 (2D4), U9.32 (2D4); no longer U10.41 (1D5), U8.41 (1D5), U9.41 (1D5)
- net iSB12: now also U10.30 (2D5), U8.30 (2D5), U9.30 (2D5); no longer U10.43 (1D4), U8.43 (1D4), U9.43 (1D4)
- net iSB13: now also U10.29 (2D6), U8.29 (2D6), U9.29 (2D6); no longer U10.44 (1D3), U8.44 (1D3), U9.44 (1D3)
- net iSB14: now also U10.27 (2D7), U8.27 (2D7), U9.27 (2D7); no longer U10.46 (1D2), U8.46 (1D2), U9.46 (1D2)
- net iSB15: now also U10.26 (2D8), U8.26 (2D8), U9.26 (2D8); no longer U10.47 (1D1), U8.47 (1D1), U9.47 (1D1)
- net iSB2: now also U10.44 (1D3), U8.44 (1D3), U9.44 (1D3); no longer U10.29 (2D6), U8.29 (2D6), U9.29 (2D6)
- net iSB3: now also U10.43 (1D4), U8.43 (1D4), U9.43 (1D4); no longer U10.30 (2D5), U8.30 (2D5), U9.30 (2D5)
- net iSB4: now also U10.41 (1D5), U8.41 (1D5), U9.41 (1D5); no longer U10.32 (2D4), U8.32 (2D4), U9.32 (2D4)
- net iSB5: now also U10.40 (1D6), U8.40 (1D6), U9.40 (1D6); no longer U10.33 (2D3), U8.33 (2D3), U9.33 (2D3)
- net iSB6: now also U10.38 (1D7), U8.38 (1D7), U9.38 (1D7); no longer U10.35 (2D2), U8.35 (2D2), U9.35 (2D2)
- net iSB7: now also U10.37 (1D8), U8.37 (1D8), U9.37 (1D8); no longer U10.36 (2D1), U8.36 (2D1), U9.36 (2D1)
- net iSB8: now also U10.36 (2D1), U8.36 (2D1), U9.36 (2D1); no longer U10.37 (1D8), U8.37 (1D8), U9.37 (1D8)
- net iSB9: now also U10.35 (2D2), U8.35 (2D2), U9.35 (2D2); no longer U10.38 (1D7), U8.38 (1D7), U9.38 (1D7)
- net at R1.1, U1.A49 (VCC1), U1.A50 (VCC1)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: now also J2.1 (VBUS)
- no-connect marks 57 -> 54
Other:
- moved on the sheet: D1, U10, U8, U9

Commit message: Today's version
Parts:
- removed J2: USB_B_Micro, symbol Connector:USB_B_Micro
- added D3, D4, D5: Led_Small, symbol device:Led_Small
- added J2, J7: Conn_01x02_Male, symbol Connector:Conn_01x02_Male
- added JP4, JP5: Jumper_NC_Small, symbol device:Jumper_NC_Small
- added R6, R7, R9: 1K, symbol Device:R_Small_US
- added R8: 10K, symbol Device:R_Small_US
- added RP7: R_PACK4, Resistor_SMD:R_Array_Convex_4x0603, symbol device:R_PACK4
Connections:
- net I2C_SCK is gone; now on net I2C_SCL: U14.JP1_7 (GPIO_04)
- net i2C_SCL is gone; now on net I2C_SCL: JP1.2, JP2.2
- net +3V3: now also U3.16 (VPU), U3.4 (VS), R8.1, RP7.5 (R4), RP7.6 (R3), RP7.7 (R2), RP7.8 (R1)
- net ExBGACK: now also U1.B48 (~{BGACK}); no longer U1.B47 (~{BG})
- net GND: now also U16.10 (DEMP), U16.11 (FLT), U16.16 (FMT), J2.2 (Pin_2), J7.2 (Pin_2), JP4.2, R6.2, R7.2, R9.2
- net I2C_SCL: now also U3.6 (SCL), U6.1 (SCLK)
- net I2C_SDA: now also U3.7 (SDA), U6.3 (SDIN/HWMODE), R8.2
- net VCC: no longer U3.4 (VS)
- net iB_AO_OE: now also U9.1 (1~{OE})
- net iCLK24M576: now also JP5.1; no longer X2.3 (OUT)
- net iEXRESET: now also U6.6 (RESETB)
- net at R1.1, U1.A49 (VCC1), U1.A50 (VCC1)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: now also J2.1 (Pin_1), J7.1 (Pin_1)
- net at U6.2 (GPO0/SWIFMODE): now also D3.2 (A)
- net at U6.4 (SDOUT/GPO2): now also D5.2 (A)
- net at U6.5 (CSB/GPO1): now also D4.2 (A)
- net at U3.10 (PV): now also RP7.4 (P4)
- net at U3.13 (TC): now also RP7.1 (P1)
- net at U3.5 (A0): now also JP4.1
- net at U3.8 (WARN): now also RP7.2 (P2)
- net at U3.9 (CRIT): now also RP7.3 (P3)
- net at TR1.4 (NC): no longer TR1.5 (NC)
- new net: JP5.2, X2.3 (OUT)
- new net: D4.1 (K), R7.1
- new net: D5.1 (K), R9.1
- new net: D3.1 (K), R6.1
- no-connect marks 54 -> 75
Other:
- moved on the sheet: C1, C10, C2, C3, C4, C5, C6, J4, J5, J6, R1, R2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

Commit message: Today's version
Parts:
- removed J3, J5, J6: Jack_3.5mm_3pin, Connector_Audio:Jack_3.5mm_Switronic_ST-005-G_horizontal, symbol w_connectors:Jack_3.5mm_3pin
- added D6, D7, D9: D_Schottky_Small, Diode_SMD:D_1206_3216Metric_Pad1.42x1.75mm_HandSolder, symbol Device:D_Schottky_Small
- added D8: D_TVS, Diode_SMD:D_1206_3216Metric_Pad1.42x1.75mm_HandSolder, symbol Device:D_TVS
- added J3, J5, J6: AudioJack3, Connector_Audio:Jack_3.5mm_Switronic_ST-005-G_horizontal, symbol Connector:AudioJack3
- added Q1, Q2: Q_PNP_BEC, Package_TO_SOT_SMD:SC-59_Handsoldering, symbol Device:Q_PNP_BEC
- added Q3, Q4, Q5, Q6: Q_NPN_BEC, Package_TO_SOT_SMD:SC-59_Handsoldering, symbol Device:Q_NPN_BEC
- added R10, R11, R12, R13, R14, R15: R_Small_US, Resistor_SMD:R_0603_1608Metric_Pad0.98x0.95mm_HandSolder, symbol Device:R_Small_US
- added U18: TLP785, Package_DIP:DIP-4_W7.62mm, symbol Isolator:TLP785
- D1, D2: footprint Diode_SMD:D_MELF_Handsoldering -> Diode_SMD:D_1206_3216Metric_Pad1.42x1.75mm_HandSolder
- D3, D4, D5: footprint (none) -> LED_SMD:LED_0603_1608Metric_Pad1.05x0.95mm_HandSolder
- J2, J7: footprint (none) -> Connector_PinHeader_2.54mm:PinHeader_1x02_P2.54mm_Vertical
- JP4: footprint (none) -> digikey-footprints:PinHeader_1x2_P2.54mm
- JP5: footprint (none) -> Jumper:SolderJumper-2_P1.3mm_Bridged_RoundedPad1.0x1.5mm
- R6, R7, R8, R9: footprint (none) -> Resistor_SMD:R_0603_1608Metric_Pad0.98x0.95mm_HandSolder
Connections:
- net +3V3: now also U18.4
- net GND: now also J3.S, Q3.2 (E), R10.2, R13.2
- net GNDA: now also J5.S
- net MIDI_IN: now also U18.3
- net MIDI_OUT: now also R11.1
- net VCC: now also Q1.2 (E), R12.1
- net at U16.6 (OUTL): now also J5.T
- net at U16.7 (OUTR): now also J5.R
- new net: D7.2 (A), J3.R
- new net: D6.1 (K), J3.T
- new net: Q3.3 (C), Q4.1 (B), R11.2
- new net: Q1.1 (B), Q2.2 (E), R12.2
- new net: Q1.3 (C), Q2.1 (B), R10.1
- new net: Q5.1 (B), Q6.2 (E), R15.1
- new net: D8.1 (A1), J6.R, Q5.2 (E), R15.2
- new net: Q3.1 (B), Q4.2 (E), R13.1
- new net: D9.1 (K), R14.1, U18.1
- new net: Q5.3 (C), Q6.1 (B), R14.2
- new net: Q6.3 (C), U18.2
- new net: D7.1 (K), Q4.3 (C)
- new net: D6.2 (A), Q2.3 (C)
- new net: D8.2 (A2), D9.2 (A), J6.T
- no-connect marks 75 -> 70
Other:
- note added: "TRS MIDI IN"
- note added: "TRS MIDI OUT"

Commit message: DRC free version
Parts:
- removed JP1: Jumper_NC_Small, digikey-footprints:PinHeader_1x2_P2.54mm, symbol device:Jumper_NC_Small
- removed JP5: Jumper_NC_Small, Jumper:SolderJumper-2_P1.3mm_Bridged_RoundedPad1.0x1.5mm, symbol device:Jumper_NC_Small
- removed TP1: TestPoint, TestPoint:TestPoint_THTPad_2.0x2.0mm_Drill1.0mm, symbol Connector:TestPoint
- removed X1: SG-8002DC(24.576MHz), Oscillator:Oscillator_SeikoEpson_SG-8002DC, symbol Oscillator:SG-8002DC
- J4: footprint Module:Raspberry_Pi_Zero_Socketed_THT_FaceDown_MountingHoles -> x68000-ext:Raspberry_Pi_Zero_Socketed_THT_FaceDown_MountingHoles
- JP4: footprint digikey-footprints:PinHeader_1x2_P2.54mm -> Jumper:SolderJumper-2_P1.3mm_Bridged_RoundedPad1.0x1.5mm
- U10: renamed from U11; footprint Housings_SSOP:SSOP-48_7.5x15.9mm_Pitch0.635mm -> x68000-ext:SSOP-48_7.5x15.9mm_Pitch0.635mm
- U17, U2: footprint Package_TO_SOT_SMD:TO-263-3_TabPin2 -> Package_TO_SOT_SMD:SOT-223-3_TabPin2
- U4, U5: footprint Housings_SSOP:SSOP-48_7.5x15.9mm_Pitch0.635mm -> x68000-ext:SSOP-48_7.5x15.9mm_Pitch0.635mm
- U6: renamed from U7; footprint Housings_SSOP:SSOP-48_7.5x15.9mm_Pitch0.635mm -> x68000-ext:SSOP-48_7.5x15.9mm_Pitch0.635mm
- U7: renamed from U8; footprint Housings_SSOP:SSOP-48_7.5x15.9mm_Pitch0.635mm -> x68000-ext:SSOP-48_7.5x15.9mm_Pitch0.635mm
- U8: renamed from U9; footprint Housings_SSOP:SSOP-48_7.5x15.9mm_Pitch0.635mm -> x68000-ext:SSOP-48_7.5x15.9mm_Pitch0.635mm
- U9: renamed from U10; footprint Housings_SSOP:SSOP-48_7.5x15.9mm_Pitch0.635mm -> x68000-ext:SSOP-48_7.5x15.9mm_Pitch0.635mm
- renumbered JP2 to JP1, U6 to U11
Connections:
- net iPCL is gone; now on net iEXPCL: U14.JP1_36 (GPIO_029)
- net +3V3: now also U10.18 (VCC), U10.31 (VCC), U4.18 (VCC), U4.31 (VCC), U5.18 (VCC), U5.31 (VCC), U6.18 (VCC), U6.31 (VCC), U7.18 (VCC), U7.31 (VCC), U8.18 (VCC), U8.31 (VCC), U9.18 (VCC), U9.31 (VCC)
- net BUS_MODE0: now also U14.JP1_18 (GPIO_013); no longer U14.JP1_20 (GPIO_015)
- net BUS_MODE1: now also U14.JP1_20 (GPIO_015); no longer U14.JP1_19 (GPIO_014)
- net BUS_MODE2: now also U14.JP1_22 (GPIO_017); no longer U14.JP1_18 (GPIO_013)
- net BUS_MODE3: now also U14.JP1_24 (GPIO_019); no longer U14.JP1_17 (GPIO_012)
- net ExHSYNC: now also U10.22 (2B7); no longer U10.20 (2B6)
- net ExVSYNC: now also U10.20 (2B6); no longer U10.22 (2B7)
- net I2C_SCL: now also IC1.13 (SCL); no longer JP1.2
- net I2C_SDA: now also JP1.2
- net I2S_BCLK: now also U14.JP1_21 (GPIO_016); no longer U14.JP1_24 (GPIO_019)
- net I2S_DATA: now also U14.JP1_17 (GPIO_012); no longer U14.JP1_22 (GPIO_017)
- net I2S_LRCK: now also U14.JP1_19 (GPIO_014); no longer U14.JP1_23 (GPIO_018)
- net I2S_MCLK: now also U14.JP1_23 (GPIO_018); no longer U14.JP1_21 (GPIO_016)
- net VCC: no longer U1.B49 (VCC1), U1.B50 (VCC1)
- net iCLK24M576: now also X2.3 (OUT)
- net iHSYNC: now also U10.27 (2A7); no longer U10.29 (2A6)
- net iVSYNC: now also U10.29 (2A6); no longer U10.27 (2A7)
- net +12V_S: now reaches R2.1, U1.A22 (+12V), U1.A23 (+12V), U3.15 (IN+2)
- net VCC2_S: now reaches R3.1, U1.A42 (VCC2), U1.A43 (VCC2), U3.2 (IN+3)
- net VCC_S: now reaches J2.1 (Pin_1), J7.1 (Pin_1), R1.1, U1.A49 (VCC1), U1.A50 (VCC1), U3.12 (IN+1)
- net VCC_S: now also U1.B49 (VCC1), U1.B50 (VCC1)
- net at RP7.2 (P2): now also U3.10 (PV); no longer U3.8 (WARN)
- net at RP7.4 (P4): now also U3.8 (WARN); no longer U3.10 (PV)
- net VCC2: now reaches R3.2, U3.1 (IN-3)
- net at D2.1 (K), U14.JP1_11 (GPIO-0_VCC_SYS): no longer U14.JP2_11 (GPIO-1_VCC_SYS)
- no-connect marks 70 -> 72
Other:
- note removed: "Alternative"
- moved on the sheet: IC1, JP1, TP4, X2

Commit message: Alpha version
Parts:
- added J8: Conn_02x07_Odd_Even, Connector_PinHeader_2.54mm:PinHeader_2x08_P2.54mm_Vertical, symbol Connector_Generic:Conn_02x08_Odd_Even
- added J9: Conn_01x02_Male, Connector_PinHeader_2.54mm:PinHeader_1x02_P2.54mm_Vertical, symbol Connector:Conn_01x02_Male
- added JP2, JP5: Jumper_NO_Small, Jumper:SolderJumper-2_P1.3mm_Open_RoundedPad1.0x1.5mm, symbol device:Jumper_NO_Small
- J3: value AudioJack3 -> MIDI OUT
- J6: value AudioJack3 -> MIDI IN
Connections:
- net FMWR is gone; now on net FM_WR: U14.JP2_31 (GPIO_124)
- net +3V3: now also J8.1 (Pin_1)
- net FM_CLK4M: now also J4.26 (GPIO7/CE1-N), J8.3 (Pin_3)
- net FM_DAT: now also J4.32 (GPIO12), J8.8 (Pin_8)
- net FM_IRQ: now also J4.29 (GPIO5), J8.4 (Pin_4)
- net FM_LRCK: now also J4.33 (GPIO13), J8.9 (Pin_9)
- net FM_PHY: now also J4.31 (GPIO6), J8.7 (Pin_7)
- net FM_RD: now also J4.27 (ID_SD), J8.6 (Pin_6)
- net FM_SCLK: now also J4.36 (GPIO16), J8.10 (Pin_10)
- net FM_SDATA: now also J4.37 (GPIO26), J8.11 (Pin_11)
- net GND: now also U3.17 (PAD), J8.15 (Pin_15), J8.16 (Pin_16)
- net I2C_SCL: now also J8.13 (Pin_13)
- net I2C_SDA: now also J8.14 (Pin_14)
- net MIDI_IN: now also JP2.2
- net MIDI_OUT: now also JP5.2
- net VCC: now also J8.2 (Pin_2), J9.1 (Pin_1); no longer J4.2 (5V), J4.4 (5V)
- net iEXRESET: now also J4.40 (GPIO21), J8.12 (Pin_12)
- net at J4.10 (GPIO15/RXD0/RXD1): now also JP5.1
- net FM_WR: now reaches J4.28 (ID_SC)
- net FM_WR: now also J8.5 (Pin_5)
- net at J4.8 (GPIO14/TXD0/TXD1): now also JP2.1
- new net: J4.2 (5V), J4.4 (5V), J9.2 (Pin_2)
- no-connect marks 72 -> 60

Commit message: current version (DE0 Nano is upside down :-( )
Parts:
- added C13, C14, C15, C16, C17, C18: 0.1uF, Capacitor_SMD:C_0603_1608Metric_Pad1.08x0.95mm_HandSolder, symbol Device:C_Small
- added C19, C20: 2.2nF, Capacitor_SMD:C_0603_1608Metric_Pad1.08x0.95mm_HandSolder, symbol Device:C_Small
- added R16, R17: 10K, Resistor_SMD:R_0603_1608Metric_Pad0.98x0.95mm_HandSolder, symbol Device:R_Small_US
Connections:
- net +3V3: now also C13.1, C14.1, C15.1, C16.1, C17.1, C18.1
- net GND: now also C13.2, C14.2, C15.2, C16.2, C17.2, C18.2
- net GNDA: now also C19.2, C20.1
- net at J5.R: now also C20.2, R17.2; no longer U16.7 (OUTR)
- net at J5.T: now also C19.1, R16.2; no longer U16.6 (OUTL)
- new net: R16.1, U16.6 (OUTL)
- new net: R17.1, U16.7 (OUTR)
