File: kepler-x.kicad_sch (KiCad schematic)
At the start: 104 parts, among them IC1 SLG46826G, J1 HDMI_C_1.3, J2 Conn_01x02_Male, J3 MIDI OUT, J4 RasPI_IO_Header_B+, J5 AudioJack3, J6 MIDI IN, J7 Conn_01x02_Male, J8 Conn_02x07_Odd_Even, J9 Conn_01x02_Male, Q1 Q_PNP_BEC, Q2 Q_PNP_BEC, Q3 Q_NPN_BEC, Q4 Q_NPN_BEC, Q5 Q_NPN_BEC, Q6 Q_NPN_BEC, SW1 SWITCH_INV, SW2 SWITCH_INV, U1 Bus-X68000-ext, U10 74LVTH162245, U11 WM8804GEDS{slash}RV, U12 TC7MPB9307F, U13 TC7MPB9307F, U14 P0082(DE0-NANO), U15 PLR135-T10, U16 PCM5102, U17 LT1117-3.3, U18 TLP785, U2 LT1117-3.3, U3 INA3221, U4 74AHC16374, U5 74AHC16374, U6 74AHC16374, U7 74AHC16374, U8 74AHC16374, U9 74AHC16374, X2 ASV-xxxMHz, Y1 12MHz

Commit message: Fix upside down foot print.
Parts:
- removed U18: TLP785, Package_DIP:DIP-4_W7.62mm, symbol Isolator:TLP785
- added R18: 10K, Resistor_SMD:R_0603_1608Metric_Pad0.98x0.95mm_HandSolder, symbol Device:R_Small_US
- added U18: H11L1, Package_DIP:DIP-6_W7.62mm, symbol Isolator:H11L1
- U14: footprint x68000-ext:MODULE_P0082_BOTTOMMOUNT -> x68000-ext:MODULE_P0082_TOPMOUNT
Connections:
- net +3V3: now also R18.1, U18.6
- net GND: now also U18.5
- net I2C_SCL: now also R18.2
- net MIDI_IN: now also U18.4
- net at D9.1 (K), R14.1: now also U18.1
- net at Q6.3 (C): now also U18.2
- net at D2.1 (K): now also U14.JP2_11 (GPIO-1_VCC_SYS); no longer U14.JP1_11 (GPIO-0_VCC_SYS)
- no-connect marks 60 -> 59
Other:
- moved on the sheet: TR1, U14A

Commit message: Fix for v1.0.0
Parts:
- added C21, C22: 0.1uF, Capacitor_SMD:C_0603_1608Metric_Pad1.08x0.95mm_HandSolder, symbol Device:C_Small
- J3, J5, J6: footprint Connector_Audio:Jack_3.5mm_Switronic_ST-005-G_horizontal -> x68000-ext:Jack_3.5mm_Switronic_ST-005-G_horizontal
Connections:
- net +3V3: now also U15.1 (VCC), C21.1
- net BUS_MODE0: now also U14.JP1_20 (GPIO_015); no longer U14.JP1_18 (GPIO_013)
- net BUS_MODE1: now also U14.JP1_19 (GPIO_014); no longer U14.JP1_20 (GPIO_015)
- net BUS_MODE2: now also U14.JP1_18 (GPIO_013); no longer U14.JP1_22 (GPIO_017)
- net BUS_MODE3: now also U14.JP1_17 (GPIO_012); no longer U14.JP1_24 (GPIO_019)
- net GND: now also C21.2, C22.2
- net I2S_BCLK: now also U14.JP1_24 (GPIO_019); no longer U14.JP1_21 (GPIO_016)
- net I2S_DATA: now also U14.JP1_22 (GPIO_017); no longer U14.JP1_17 (GPIO_012)
- net I2S_LRCK: now also U14.JP1_23 (GPIO_018); no longer U14.JP1_19 (GPIO_014)
- net I2S_MCLK: now also U14.JP1_21 (GPIO_016); no longer U14.JP1_23 (GPIO_018)
- net VCC: now also C22.1; no longer U15.1 (VCC)

Commit message: Ver 1.0.0 RC1
Parts:
- added D10: D_TVS, Diode_SMD:D_1206_3216Metric_Pad1.42x1.75mm_HandSolder, symbol Device:D_TVS
- J1: footprint digikey-footprints:HDMI_Mini_Female_2001-1-2-21-00-BK -> x68000-ext:HDMI_Mini_Female_DC2R019JA7
- R16, R17: value 10K -> 470
- RP1, RP2, RP3, RP4, RP7: value R_PACK4 -> 4.7k
- U17, U2: value LT1117-3.3 -> LM1117GS-3.3
- X1: renamed from X2; value ASV-xxxMHz -> ASV-24.576MHz
Connections:
- net at D7.2 (A), J3.R: now also D10.2 (A2)
- net at D6.1 (K), J3.T: now also D10.1 (A1)
