File: main/kepler-x.kicad_sch (KiCad schematic)
At the start: 139 parts, among them IC1 SLG46826G, J1 HDMI_C_1.3, J10 Conn_01x04, J11 Micro_SD_Card_Det_Hirose_DM3AT, J2 Conn_01x02_Male, J3 MIDI OUT, J4 RasPI_IO_Header_B+, J5 AudioJack3, J6 MIDI IN, J7 Conn_01x02_Male, J8 Conn_02x05_Odd_Even, J9 Conn_01x02_Male, Q1 Q_PNP_BEC, Q2 Q_PNP_BEC, Q3 Q_NPN_BEC, Q4 Q_NPN_BEC, Q5 Q_NPN_BEC, Q6 Q_NPN_BEC, SW1 SWITCH_INV, SW2 SWITCH_INV, U1 Bus-X68000-ext, U10 74LVTH162245, U11 WM8804GEDS{slash}RV, U12 TC7MPB9307F, U13 TC7MPB9307F, U14 P0082(DE0-NANO), U15 PLR135-T10, U16 PCM5102, U17 XC6201P332MR-G, U18 H11L1, U19 TC7MPB9307F, U2 LM1117GS-3.3, U20 TC7MPB9307F, U21 XC6201P332MR-G, U22 PCA9515DP, U23 74LVC541A, U3 INA3221, U4 74AHC16374, U5 74AHC16374, U6 74AHC16374, U7 74AHC16374, U8 74AHC16374, U9 74AHC16374, X1 ASV-24.576MHz, Y1 12MHz

Commit message: v2.0.0 RC1
Parts:
- removed U16: PCM5102, Package_SO:TSSOP-20_4.4x6.5mm_P0.65mm, symbol Audio:PCM5102
- added C31, C32, C34: 10uF, Capacitor_Tantalum_SMD:CP_EIA-3216-18_Kemet-A, symbol Device:C_Polarized_Small_US
- added C33: 0.1uF, Capacitor_SMD:C_0603_1608Metric_Pad1.08x0.95mm_HandSolder, symbol Device:C_Small
- added J12: Filter Sel, Connector_PinHeader_2.54mm:PinHeader_1x02_P2.54mm_Vertical, symbol Connector:Conn_01x02_Male
- added JP10: Jumper_NC_Small, Connector_PinHeader_2.54mm:PinHeader_1x02_P2.54mm_Vertical, symbol device:Jumper_NC_Small
- added JP11: Jumper_NO_Small, Jumper:SolderJumper-2_P1.3mm_Open_RoundedPad1.0x1.5mm, symbol device:Jumper_NO_Small
- added R25: 18k, Resistor_SMD:R_0603_1608Metric_Pad0.98x0.95mm_HandSolder, symbol Device:R_Small_US
- added R26: 33k, Resistor_SMD:R_0603_1608Metric_Pad0.98x0.95mm_HandSolder, symbol Device:R_Small_US
- added R27: 10K, Resistor_SMD:R_0603_1608Metric_Pad0.98x0.95mm_HandSolder, symbol Device:R_Small_US
- added TP1, TP4, TP5: GND, TestPoint:TestPoint_THTPad_2.0x2.0mm_Drill1.0mm, symbol Connector:TestPoint
- added TP6: GNDA, TestPoint:TestPoint_THTPad_2.0x2.0mm_Drill1.0mm, symbol Connector:TestPoint
- added U16: PCM5102A, Package_SO:TSSOP-20_4.4x6.5mm_P0.65mm, symbol x68000-ext:PCM5102A
- C1: footprint Capacitor_THT:CP_Radial_D5.0mm_P2.50mm -> Capacitor_Tantalum_SMD:CP_EIA-3216-18_Kemet-A
- C2: footprint Capacitor_THT:CP_Radial_D5.0mm_P2.50mm -> Capacitor_Tantalum_SMD:CP_EIA-3528-21_Kemet-B
- D10, D8: footprint Diode_SMD:D_1206_3216Metric_Pad1.42x1.75mm_HandSolder -> Diode_SMD:D_0603_1608Metric_Pad1.05x0.95mm_HandSolder
- JP1: footprint digikey-footprints:PinHeader_1x2_P2.54mm -> Connector_PinHeader_2.54mm:PinHeader_1x02_P2.54mm_Vertical
- U3: footprint Housings_DFN_QFN:QFN-16-1EP_4x4mm_Pitch0.65mm -> x68000-ext:QFN-16-1EP_4x4mm_Pitch0.65mm_with_hole
Connections:
- net +3.3VA: now also C33.1, C34.1, U16.1 (CPVDD), U16.8 (AVDD)
- net +3V3: now also C31.1, R27.1, U16.20 (DVDD)
- net GND: now also C10.1, C31.2, C32.2, J12.2 (Pin_2), R26.1, TP1.1, TP4.1, TP5.1, U16.10 (DEMP), U16.16 (FMT), U16.19 (DGND); no longer C10.2, C8.2
- net GNDA: now also C8.1, C33.2, C34.2, TP6.1, U16.3 (CPGND), U16.9 (AGND)
- net I2C_SCL: now also JP1.1; no longer J4.5 (GPIO1-R1/GPIO3-R2/SCL0/SCL1), U22.2 (SCL0)
- net I2C_SDA: now also IC1.12 (SDA), JP10.1; no longer J4.3 (GPIO0-R1/GPIO2-R2/SDA0/SDA1), JP1.2, U22.3 (SDA0)
- net I2S_BCLK: now also U16.13 (BCK)
- net I2S_DATA: now also U16.14 (DIN)
- net I2S_LRCK: now also U16.15 (LRCK)
- net I2S_MCLK: now also JP11.1
- net VCC: now also R25.2
- net AUDIO_R: now reaches C20.2, J5.R, R17.2
- net AUDIO_L: now reaches C19.1, J5.T, R16.2
- net at R16.1: now also U16.6 (OUTL)
- net at C9.1: now also U16.4 (CAPM)
- net at C9.2: now also U16.2 (CAPP)
- net at R17.1: now also U16.7 (OUTR)
- new net: C10.2, C32.1, U16.18 (LDOO)
- new net: R25.1, R26.2, U16.17 (XSMT)
- new net: J12.1 (Pin_1), R27.2, U16.11 (FLT)
- new net: JP11.2, U16.12 (SCK)
- new net: C8.2, U16.5 (VNEG)
- new net I2C_SCL_PI: J4.5 (GPIO1-R1/GPIO3-R2/SCL0/SCL1), JP1.2, U22.2 (SCL0)
- new net I2C_SDA_PI: J4.3 (GPIO0-R1/GPIO2-R2/SDA0/SDA1), JP10.2, U22.3 (SDA0)
- no-connect marks 74 -> 73
Other:
- moved on the sheet: C10, C19, C20, C7, C8, C9, J5, R16, R17, R18, R8

Commit message: v2.0.0 RC2
Parts:
- added C35: 10uF, Capacitor_Tantalum_SMD:CP_EIA-3216-18_Kemet-A, symbol Device:C_Polarized_Small_US
Connections:
- net +3V3: now also C35.1
- net GND: now also C35.2
Changed lines of the file:
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@@
     (stroke (width 0) (type default) (color 0 0 0 0))
   )
+  (wire (pts (xy 179.07 487.68) (xy 179.07 490.22))
+    (stroke (width 0) (type default) (color 0 0 0 0))
+  )
   (bus (pts (xy 168.91 266.7) (xy 168.91 269.24))
     (stroke (width 0) (type default) (color 0 0 0 0))
@@
     (stroke (width 0) (type default) (color 0 0 0 0))
   )
+  (wire (pts (xy 179.07 495.3) (xy 179.07 497.84))
+    (stroke (width 0) (type default) (color 0 0 0 0))
+  )
   (wire (pts (xy 157.48 416.56) (xy 157.48 490.22))
     (stroke (width 0) (type default) (color 0 0 0 0))
@@
     (pin "1")
   )
+  (symbol (lib_id "power:+3.3V") (at 179.07 487.68 0) (unit 1)
+    (in_bom yes) (on_board yes)
+    (property "Reference" "#PWR095" (id 0) (at 179.07 491.49 0)
+      (effects (font (size 1.27 1.27)) hide)
+    )
+    (property "Value" "+3.3V" (id 1) (at 179.07 483.235 0))
+    (property "Footprint" "" (id 2) (at 179.07 487.68 0)
+      (effects (font (size 1.27 1.27)) hide)
+    )
+    (property "Datasheet" "" (id 3) (at 179.07 487.68 0)
+      (effects (font (size 1.27 1.27)) hide)
+    )
+    (pin "1")
+  )
   (symbol (lib_id "Device:C_Small") (at 533.4 252.73 0) (unit 1)
     (in_bom yes) (on_board yes) (fields_autoplaced)
@@
     (pin "1")
   )
+  (symbol (lib_id "power:GND") (at 179.07 497.84 0) (unit 1)
+    (in_bom yes) (on_board yes) (fields_autoplaced)
+    (property "Reference" "#PWR096" (id 0) (at 179.07 504.19 0)
+      (effects (font (size 1.27 1.27)) hide)
+    )
+    (property "Value" "GND" (id 1) (at 179.07 502.285 0))
+    (property "Footprint" "" (id 2) (at 179.07 497.84 0)
+      (effects (font (size 1.27 1.27)) hide)
+    )
+    (property "Datasheet" "" (id 3) (at 179.07 497.84 0)
+      (effects (font (size 1.27 1.27)) hide)
+    )
+    (pin "1")
+  )
   (symbol (lib_id "power:GND") (at 469.9 307.34 0) (unit 1)
     (in_bom yes) (on_board yes) (fields_autoplaced)
@@
     (pin "1")
   )
+  (symbol (lib_id "Device:C_Polarized_Small_US") (at 179.07 492.76 0) (unit 1)
+    (in_bom yes) (on_board yes) (fields_autoplaced)
+    (property "Reference" "C35" (id 0) (at 181.61 491.0581 0)
+      (effects (font (size 1.27 1.27)) (justify left))
+    )
+    (property "Value" "10uF" (id 1) (at 181.61 493.5981 0)
+      (effects (font (size 1.27 1.27)) (justify left))
+    )
+    (property "Footprint" "Capacitor_Tantalum_SMD:CP_EIA-3216-18_Kemet-A" (id 2) (at 179.07 492.76 0)
+      (effects (font (size 1.27 1.27)) hide)
+    )
+    (property "Datasheet" "~" (id 3) (at 179.07 492.76 0)
+      (effects (font (size 1.27 1.27)) hide)
+    )
+    (pin "1")
+    (pin "2")
+  )
   (symbol (lib_id "power:GNDA") (at 579.755 320.04 0) (unit 1)
     (in_bom yes) (on_board yes) (fields_autoplaced)
@@
   )
   (symbol (lib_id "power:+3.3V") (at 166.37 487.68 0) (unit 1)
-    (in_bom yes) (on_board yes) (fields_autoplaced)
+    (in_bom yes) (on_board yes)
     (property "Reference" "#PWR055" (id 0) (at 166.37 491.49 0)
       (effects (font (size 1.27 1.27)) hide)
     )
-    (property "Value" "+3.3V" (id 1) (at 166.37 481.965 0))
+    (property "Value" "+3.3V" (id 1) (at 166.37 483.235 0))
     (property "Footprint" "" (id 2) (at 166.37 487.68 0)
       (effects (font (size 1.27 1.27)) hide)
@@
       (reference "#PWR094") (unit 1) (value "GNDA") (footprint "")
     )
+    (path "/33611cbd-bda3-4485-a6b4-4ad6e8799f89"
+      (reference "#PWR095") (unit 1) (value "+3.3V") (footprint "")
+    )
+    (path "/53c550a3-77bc-42cd-99e5-01643159eb4c"
+      (reference "#PWR096") (unit 1) (value "GND") (footprint "")
+    )
     (path "/17546b8e-7f29-4d68-968f-e270ca497b3c"
       (reference "#PWR0101") (unit 1) (value "GND") (footprint "")
@@
       (reference "C34") (unit 1) (value "10uF") (footprint "Capacitor_Tantalum_SMD:CP_EIA-3216-18_Kemet-A")
     )
+    (path "/b18a9a7d-d1a6-47bc-9fac-7514e615b3d1"
+      (reference "C35") (unit 1) (value "10uF") (footprint "Capacitor_Tantalum_SMD:CP_EIA-3216-18_Kemet-A")
+    )
     (path "/949b3f55-bccf-4df9-aa1d-218db6fa6e70"

Commit message: 3.5mmジャックの Tipと Ringが逆になっていた問題などを修正
Parts:
- removed JP11: Jumper_NO_Small, Jumper:SolderJumper-2_P1.3mm_Open_RoundedPad1.0x1.5mm, symbol device:Jumper_NO_Small
- added JP11: SolderJumper_3_Bridged12, Jumper:SolderJumper-3_P1.3mm_Bridged12_RoundedPad1.0x1.5mm, symbol Jumper:SolderJumper_3_Bridged12
- D1, D2, D6, D7, D9: value D_Schottky_Small -> CUHS20S30
- J1: footprint x68000-ext:HDMI_Mini_Female_DC2R019JA7 -> digikey-footprints:HDMI_Mini_Female_2001-1-2-21-00-BK
- J3, J5, J6: footprint Connector_Audio:Jack_3.5mm_CUI_SJ-3524-SMT_Horizontal -> x68000-ext:AudioJack_3.5_pj313d-smt; symbol Connector:AudioJack3 -> x68000-ext:AudioJack3_PJ313D
- Q1, Q2: value Q_PNP_BEC -> 2SA1162GR
- Q3, Q4, Q5, Q6: value Q_NPN_BEC -> 2SC2712GR
- R18, R8: value 10K -> 10k
- R4, R5: value R_US -> 10k
- U3: footprint x68000-ext:QFN-16-1EP_4x4mm_Pitch0.65mm_with_hole -> Housings_DFN_QFN:QFN-16-1EP_4x4mm_Pitch0.65mm
- Y1: value 12MHz -> XJHCELNANF-12MHZ
Connections:
- net AUDIO_L: now also J5.3 (Tip); no longer J5.T
- net AUDIO_R: now also J5.2 (Ring); no longer J5.R
- net GND: now also J3.1 (Sleeve), JP11.2 (C); no longer J3.S
- net GNDA: now also J5.1 (Sleeve); no longer J5.S
- net I2S_MCLK: now also JP11.3 (B)
- net at D10.1 (A1), D6.1 (K): now also J3.2 (Ring); no longer J3.R
- net at D10.2 (A2), D7.2 (A): now also J3.3 (Tip); no longer J3.T
- net at D8.1 (A1), Q5.2 (E), R15.2: now also J6.3 (Tip); no longer J6.T
- net at U16.12 (SCK): now also JP11.1 (A)
- net at D8.2 (A2), D9.2 (A): now also J6.2 (Ring); no longer J6.R
- no-connect marks 73 -> 72

Commit message: 再再度出し直し(v2.0.2)
Parts:
- D11, D3, D4, D5: LCSC (none) -> C72043
- J3, J5, J6: LCSC (none) -> C668608
- RP1, RP2, RP3, RP4, RP7: LCSC (none) -> C700514
- RP10: LCSC (none) -> C327045
- RP5, RP6: LCSC (none) -> C425067
- RP8, RP9: LCSC (none) -> C779384
- U18: footprint Package_DIP:SMDIP-6_W7.62mm -> Package_DIP:SMDIP-6_W9.53mm; LCSC (none) -> C78589
- U22: footprint Package_SO:SOP-8_5.28x5.23mm_P1.27mm -> Housings_SSOP:TSSOP-8_3x3mm_Pitch0.65mm; LCSC (none) -> C129512
Changed lines of the file:
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@@
       (effects (font (size 1.27 1.27)) hide)
     )
+    (property "LCSC" "C668608" (id 4) (at 539.75 441.96 0)
+      (effects (font (size 1.27 1.27)) hide)
+    )
     (pin "1")
     (pin "2")
@@
       (effects (font (size 1.27 1.27)) hide)
     )
-    (property "Datasheet" "" (id 3) (at 273.05 347.98 0))
+    (property "Datasheet" "https://jlcpcb.com/partdetail/Yageo-YC164_FR074K7L/C700514" (id 3) (at 273.05 347.98 0))
+    (property "LCSC" "C700514" (id 4) (at 273.05 347.98 0)
+      (effects (font (size 1.27 1.27)) hide)
+    )
     (pin "1")
     (pin "2")
@@
       (effects (font (size 1.27 1.27)) hide)
     )
-    (property "Datasheet" "" (id 3) (at 283.21 490.22 0))
+    (property "Datasheet" "https://jlcpcb.com/partdetail/Yageo-YC164_FR074K7L/C700514" (id 3) (at 283.21 490.22 0))
+    (property "LCSC" "C700514" (id 4) (at 283.21 490.22 0)
+      (effects (font (size 1.27 1.27)) hide)
+    )
     (pin "1")
     (pin "2")
@@
       (effects (font (size 1.27 1.27)) hide)
     )
-    (property "Datasheet" "" (id 3) (at 751.84 368.3 90))
+    (property "Datasheet" "https://jlcpcb.com/partdetail/EverlightElec-19_217_GHC_YR1S23T/C72043" (id 3) (at 751.84 368.3 90))
+    (property "LCSC" "C72043" (id 4) (at 751.84 368.3 0)
+      (effects (font (size 1.27 1.27)) hide)
+    )
     (pin "1")
     (pin "2")
@@
       (effects (font (size 1.27 1.27)) hide)
     )
-    (property "Datasheet" "" (id 3) (at 273.05 490.22 0))
+    (property "Datasheet" "https://jlcpcb.com/partdetail/Yageo-YC164_FR074K7L/C700514" (id 3) (at 273.05 490.22 0))
+    (property "LCSC" "C700514" (id 4) (at 273.05 490.22 0)
+      (effects (font (size 1.27 1.27)) hide)
+    )
     (pin "1")
     (pin "2")
@@
       (effects (font (size 1.27 1.27)) hide)
     )
-    (property "Datasheet" "" (id 3) (at 732.155 330.2 0))
+    (property "Datasheet" "https://jlcpcb.com/partdetail/Yageo-YC164_JR0747RL/C327045" (id 3) (at 732.155 330.2 0))
+    (property "LCSC" "C327045" (id 4) (at 732.155 330.2 0)
+      (effects (font (size 1.27 1.27)) hide)
+    )
     (pin "1")
     (pin "2")
@@
       (effects (font (size 1.27 1.27)) hide)
     )
-    (property "Datasheet" "" (id 3) (at 711.2 317.5 0))
+    (property "Datasheet" "https://jlcpcb.com/partdetail/Yageo-YC164_JR0747KL/C779384" (id 3) (at 711.2 317.5 0))
+    (property "LCSC" "C779384" (id 4) (at 711.2 317.5 0)
+      (effects (font (size 1.27 1.27)) hide)
+    )
     (pin "1")
     (pin "2")
@@
       (effects (font (size 1.27 1.27)) hide)
     )
+    (property "LCSC" "C668608" (id 4) (at 597.535 309.88 0)
+      (effects (font (size 1.27 1.27)) hide)
+    )
     (pin "1")
     (pin "2")
@@
       (effects (font (size 1.27 1.27)) hide)
     )
-    (property "Datasheet" "" (id 3) (at 344.805 43.18 0))
+    (property "Datasheet" "https://jlcpcb.com/partdetail/418803-4D03WGJ0271T5E/C425067" (id 3) (at 344.805 43.18 0))
+    (property "LCSC" "C425067" (id 4) (at 344.805 43.18 0)
+      (effects (font (size 1.27 1.27)) hide)
+    )
     (pin "1")
     (pin "2")
@@
       (effects (font (size 1.27 1.27)) hide)
     )
-    (property "Datasheet" "" (id 3) (at 283.21 347.98 0))
+    (property "Datasheet" "https://jlcpcb.com/partdetail/Yageo-YC164_FR074K7L/C700514" (id 3) (at 283.21 347.98 0))
+    (property "LCSC" "C700514" (id 4) (at 283.21 347.98 0)
+      (effects (font (size 1.27 1.27)) hide)
+    )
     (pin "1")
     (pin "2")
@@
       (effects (font (size 1.27 1.27)) hide)
     )
-    (property "Datasheet" "" (id 3) (at 85.09 191.77 0))
+    (property "Datasheet" "https://jlcpcb.com/partdetail/Yageo-YC164_FR074K7L/C700514" (id 3) (at 85.09 191.77 0))
+    (property "LCSC" "C700514" (id 4) (at 85.09 191.77 0)
+      (effects (font (size 1.27 1.27)) hide)
+    )
     (pin "1")
     (pin "2")
@@
       (effects (font (size 1.27 1.27)) hide)
     )
-    (property "Datasheet" "" (id 3) (at 388.62 257.81 90))
+    (property "Datasheet" "https://jlcpcb.com/partdetail/EverlightElec-19_217_GHC_YR1S23T/C72043" (id 3) (at 388.62 261.62 90))
+    (property "LCSC" "C72043" (id 4) (at 388.62 257.81 90)
+      (effects (font (size 1.27 1.27)) hide)
+    )
     (pin "1")
     (pin "2")
@@
     (property "Reference" "U18" (id 0) (at 641.35 432.435 0))
     (property "Value" "H11L1" (id 1) (at 641.35 434.975 0))
-    (property "Footprint" "Package_DIP:SMDIP-6_W7.62mm" (id 2) (at 628.904 436.88 0)
+    (property "Footprint" "Package_DIP:SMDIP-6_W9.53mm" (id 2) (at 628.904 436.88 0)
       (effects (font (size 1.27 1.27)) hide)
     )
-    (property "Datasheet" "https://www.onsemi.com/pub/Collateral/H11L3M-D.PDF" (id 3) (at 628.904 436.88 0)
+    (property "Datasheet" "https://jlcpcb.com/partdetail/EverlightElec-H11L1S_TA/C78589" (id 3) (at 628.904 436.88 0)
+      (effects (font (size 1.27 1.27)) hide)
+    )
+    (property "LCSC" "C78589" (id 4) (at 631.19 436.88 0)
       (effects (font (size 1.27 1.27)) hide)
     )
@@
       (effects (font (size 1.27 1.27)) hide)
     )
-    (property "Datasheet" "" (id 3) (at 396.24 257.81 90))
+    (property "Datasheet" "https://jlcpcb.com/partdetail/EverlightElec-19_217_GHC_YR1S23T/C72043" (id 3) (at 396.24 257.81 90))
+    (property "LCSC" "C72043" (id 4) (at 396.24 257.81 90)
+      (effects (font (size 1.27 1.27)) hide)
+    )
     (pin "1")
     (pin "2")
@@
       (effects (font (size 1.27 1.27)) hide)
     )
-    (property "Datasheet" "" (id 3) (at 726.44 317.5 0))
+    (property "Datasheet" "https://jlcpcb.com/partdetail/Yageo-YC164_JR0747KL/C779384" (id 3) (at 726.44 317.5 0))
+    (property "LCSC" "C779384" (id 4) (at 726.44 317.5 0)
+      (effects (font (size 1.27 1.27)) hide)
+    )
     (pin "1")
     (pin "2")
@@
       (effects (font (size 1.27 1.27)) (justify left))
     )
-    (property "Footprint" "Package_SO:SOP-8_5.28x5.23mm_P1.27mm" (id 2) (at 695.96 195.58 0)
+    (property "Footprint" "Housings_SSOP:TSSOP-8_3x3mm_Pitch0.65mm" (id 2) (at 695.96 195.58 0)
+      (effects (font (size 1.27 1.27)) hide)
+    )
+    (property "Datasheet" "https://jlcpcb.com/partdetail/NxpSemicon-PCA9515DP/C129512" (id 3) (at 665.48 229.87 0)
       (effects (font (size 1.27 1.27)) hide)
     )
-    (property "Datasheet" "http://www.nxp.com/documents/data_sheet/PCA9536.pdf" (id 3) (at 665.48 229.87 0)
+    (property "LCSC" "C129512" (id 4) (at 670.56 186.69 0)
       (effects (font (size 1.27 1.27)) hide)
     )
@@
       (effects (font (size 1.27 1.27)) hide)
     )
-    (property "Datasheet" "" (id 3) (at 392.43 257.81 90))
+    (property "Datasheet" "https://jlcpcb.com/partdetail/EverlightElec-19_217_GHC_YR1S23T/C72043" (id 3) (at 392.43 257.81 90))
+    (property "LCSC" "C72043" (id 4) (at 392.43 257.81 90)
+      (effects (font (size 1.27 1.27)) hide)
+    )
     (pin "1")
     (pin "2")
@@
       (effects (font (size 1.27 1.27)) hide)
     )
+    (property "LCSC" "C668608" (id 4) (at 577.85 441.96 0)
+      (effects (font (size 1.27 1.27)) hide)
+    )
     (pin "1")
     (pin "2")
@@
       (effects (font (size 1.27 1.27)) hide)
     )
-    (property "Datasheet" "" (id 3) (at 344.805 53.34 0))
+    (property "Datasheet" "https://jlcpcb.com/partdetail/418803-4D03WGJ0271T5E/C425067" (id 3) (at 344.805 53.34 0))
+    (property "LCSC" "C425067" (id 4) (at 344.805 53.34 0)
+      (effects (font (size 1.27 1.27)) hide)
+    )
     (pin "1")
     (pin "2")
@@
     )
     (path "/982c421f-1f8b-403b-85e2-a0b1beb0d514"
-      (reference "U18") (unit 1) (value "H11L1") (footprint "Package_DIP:SMDIP-6_W7.62mm")
+      (reference "U18") (unit 1) (value "H11L1") (footprint "Package_DIP:SMDIP-6_W9.53mm")
     )
     (path "/0b5ed3b7-3cc4-4866-8c2e-fe4a84aa15be"
@@
     )
     (path "/b81e17be-bed4-4b3f-8573-6613b6f56621"
-      (reference "U22") (unit 1) (value "PCA9515DP") (footprint "Package_SO:SOP-8_5.28x5.23mm_P1.27mm")
+      (reference "U22") (unit 1) (value "PCA9515DP") (footprint "Housings_SSOP:TSSOP-8_3x3mm_Pitch0.65mm")
     )
     (path "/65f3f2f1-b07b-49ee-a85b-3048b308213e"

Commit message: 現状をコミット
Parts:
- added C?: 0.1uF, Capacitor_SMD:C_0603_1608Metric_Pad1.08x0.95mm_HandSolder, symbol Device:C_Small
- added R? (x2): 10K, Resistor_SMD:R_0603_1608Metric_Pad0.98x0.95mm_HandSolder, symbol Device:R_Small_US
Connections:
- net +3V3: now also C?.1
- net GND: now also J11.10 (DET_A), JP11.1 (A), U4.26 (2D8), U4.27 (2D7), U4.29 (2D6), U4.30 (2D5), U4.32 (2D4), U5.47 (1D1), C?.2, R?.2, R?.2; no longer JP11.2 (C), U23.19 (~{G2})
- net MMC_SCK: no longer U23.5 (A4)
- net WM8804_INTn: now also R?.1
- net at U23.15 (Y4): now also D11.2 (A); no longer J11.10 (DET_A)
- net at J11.9 (DET_B): now also RP8.1 (P1), U23.19 (~{G2}); no longer D11.2 (A)
- net at D4.2 (A), U11.5 (CSB/GPO1): now also R?.1
- net at U16.12 (SCK): now also JP11.2 (C); no longer JP11.1 (A)
- new net MMC_ACCESS: U23.5 (A4)
- no-connect marks 72 -> 65
Other:
- moved on the sheet: C10, C3, C31, C32, C7, D11, D3, D4, J12, JP11, JP7, R24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

Commit message: 現状をコミット
Parts:
- removed JP1, JP10: Jumper_NC_Small, Connector_PinHeader_2.54mm:PinHeader_1x02_P2.54mm_Vertical, symbol device:Jumper_NC_Small
- removed SW1, SW2: SWITCH_INV, Pin_Headers:Pin_Header_Straight_1x03, symbol device:SWITCH_INV
- added D12: SS2040FL, Diode_SMD:D_1206_3216Metric_Pad1.42x1.75mm_HandSolder, symbol device:D_Schottky_Small
- added R30, R31: 10k, Resistor_SMD:R_0603_1608Metric_Pad0.98x0.95mm_HandSolder, symbol Device:R_Small_US
- added SW1: SW_DPDT_x2, x68000-ext:MST22D18G2-SlideSwitch-DPDT, symbol Switch:SW_DPDT_x2
- added SW3: SW_DIP_x02, Button_Switch_SMD:SW_DIP_SPSTx02_Slide_KingTek_DSHP02TS_W7.62mm_P1.27mm, symbol Switch:SW_DIP_x02
- added TP7: FPGA_5V, TestPoint:TestPoint_THTPad_2.0x2.0mm_Drill1.0mm, symbol Connector:TestPoint
- added TP8: FPGA_3V3, TestPoint:TestPoint_THTPad_2.0x2.0mm_Drill1.0mm, symbol Connector:TestPoint
- D1, D2, D6, D7, D9: value CUHS20S30 -> SS2040FL
- FB1, FB2, FB3: value BK2125HS750-T -> BLM18AG121SN1D; LCSC (none) -> C76892
- R28, R29: renamed from R?; value 10K -> 4.7K
- U1: footprint x68000-ext:x68000-ext-cardedge -> x68000-ext:x68000-ext-cardedge-fit-with-pad
- U10: value 74LVTH162245 -> 74LVCR162245; footprint x68000-ext:SSOP-48_7.5x15.9mm_Pitch0.635mm -> Package_SO:TSSOP-48_6.1x12.5mm_P0.5mm; LCSC (none) -> C7039
- U4, U5, U6, U7, U8, U9: value 74AHC16374 -> 74LVC16374; footprint x68000-ext:SSOP-48_7.5x15.9mm_Pitch0.635mm -> Package_SO:TSSOP-48_6.1x12.5mm_P0.5mm; LCSC (none) -> C7665
- gave numbers to parts that had none: 1
Connections:
- net +3V3: now also R30.1, R31.1
- net ExIACK2: now also SW1.4 (A)
- net ExIACK4: now also SW1.6 (C)
- net ExIRQ2: now also SW1.1 (A)
- net ExIRQ4: now also SW1.3 (C)
- net I2C_SCL: now also SW3.1
- net I2C_SCL_EX: now also R30.2
- net I2C_SCL_PI: now also SW3.4
- net I2C_SDA: now also SW3.2
- net I2C_SDA_EX: now also R31.2
- net I2C_SDA_PI: now also SW3.3
- net VCC: now also D12.1 (K)
- net iAS: now also U10.2 (1B1); no longer IC1.15 (IO4)
- net iIACK: now also U10.37 (1A8); no longer U10.35 (2A2)
- net at U12.16 (B3), U19.13 (B6): now also SW1.2 (B)
- net at U10.12 (1B8): now also SW1.5 (B)
- net iAS_BUF: now reaches U10.47 (1A1)
- net iAS_BUF: now also IC1.15 (IO4)
- net at D2.1 (K), U14.JP2_11 (GPIO-1_VCC_SYS): now also D12.2 (A)
- net at U14.JP1_11 (GPIO-0_VCC_SYS): now also TP7.1
- net at U14.JP1_29 (GPIO-0_VCC3P3): now also TP8.1
- no-connect marks 65 -> 61
Other:
- moved on the sheet: C13, C35, D2
