File: main/kepler-x.kicad_sch (KiCad schematic)
At the start: 160 parts, among them IC1 SLG46826G, J1 HDMI_C_1.3, J10 Conn_01x04, J11 Micro_SD_Card_Det_Hirose_DM3AT, J12 Filter Sel, J2 Conn_01x02_Male, J3 MIDI OUT, J4 RasPI_IO_Header_B+, J5 AudioJack3, J6 MIDI IN, J7 Conn_01x02_Male, J8 Conn_02x05_Odd_Even, J9 Conn_01x02_Male, Q1 2SA1162GR, Q2 2SA1162GR, Q3 2SC2712GR, Q4 2SC2712GR, Q5 2SC2712GR, Q6 2SC2712GR, SW1 SW_DPDT_x2, SW3 SW_DIP_x02, U1 Bus-X68000-ext, U10 74LVCR162245, U11 WM8804GEDS{slash}RV, U12 TC7MPB9307F, U13 TC7MPB9307F, U14 P0082(DE0-NANO), U15 PLR135-T10, U16 PCM5102A, U17 XC6201P332MR-G, U18 H11L1, U19 TC7MPB9307F, U2 LM1117GS-3.3, U20 TC7MPB9307F, U21 XC6201P332MR-G, U22 PCA9515DP, U23 74LVC541A, U3 INA3221, U4 74LVC16374, U5 74LVC16374, U6 74LVC16374, U7 74LVC16374, U8 74LVC16374, U9 74LVC16374, X1 ASV-24.576MHz, Y1 XJHCELNANF-12MHZ

Commit message: V3.0.0
Parts:
- removed D11: Led_Small, LED_SMD:LED_0603_1608Metric_Pad1.05x0.95mm_HandSolder, symbol device:Led_Small
- removed JP3: Jumper_NC_Small, Jumper:SolderJumper-2_P1.3mm_Bridged_RoundedPad1.0x1.5mm, symbol device:Jumper_NC_Small
- removed JP7: SolderJumper_3_Bridged12, Jumper:SolderJumper-3_P1.3mm_Bridged12_RoundedPad1.0x1.5mm, symbol Jumper:SolderJumper_3_Bridged12
- added C37, C38: 0.1uF, Capacitor_SMD:C_0603_1608Metric_Pad1.08x0.95mm_HandSolder, symbol Device:C_Small
- added J13, J14: Conn_01x02_Pin, Connector_PinHeader_2.54mm:PinHeader_1x02_P2.54mm_Vertical, symbol Connector:Conn_01x02_Pin
- added JP1, JP10: SolderJumper_3_Bridged12, Jumper:SolderJumper-3_P1.3mm_Bridged12_RoundedPad1.0x1.5mm, symbol Jumper:SolderJumper_3_Bridged12
- added LED1, LED2: WS2812C, x68000-ext:WM2812C-2020, symbol x68000-ext:WS2812C
- added NT1: NetTie_2, NetTie:NetTie-2_THT_Pad1.0mm, symbol Device:NetTie_2
- added R32: 10k, Resistor_SMD:R_0603_1608Metric_Pad0.98x0.95mm_HandSolder, symbol Device:R_Small_US
- added SP1: SPEAKER, x68000-ext:UGCT7525AN4, symbol device:SPEAKER
- added U24: CH32V003F4P6, Package_SO:TSSOP-20_4.4x6.5mm_P0.65mm, symbol x68000-ext:CH32V003A4M6
- C1, C31, C32, C34, C35: LCSC (none) -> C128254
- C2: LCSC (none) -> C129567
- D10, D8: LCSC (none) -> C98320
- J10, J8: now left out of the parts list
- J12: footprint Connector_PinHeader_2.54mm:PinHeader_1x02_P2.54mm_Vertical -> Jumper:SolderJumper-2_P1.3mm_Open_RoundedPad1.0x1.5mm; symbol Connector:Conn_01x02_Male -> Jumper:SolderJumper_2_Open
- J2, J7, J9: value Conn_01x02_Male -> Conn_01x02_Pin; symbol Connector:Conn_01x02_Male -> Connector:Conn_01x02_Pin
- J4: value RasPI_IO_Header_B+ -> Raspberry Pi; LCSC (none) -> C2977589
- Q1, Q2: footprint Package_TO_SOT_SMD:SC-59_Handsoldering -> x68000-ext:SC-59_Handsoldering; LCSC (none) -> C155455
- Q3, Q4, Q5, Q6: value 2SC2712GR -> 2SC2712-GR; footprint Package_TO_SOT_SMD:SC-59_Handsoldering -> x68000-ext:SC-59_Handsoldering; LCSC (none) -> C83447
- R2, R3: value R100 (0.1Ω, 0.1W) -> 1R; LCSC C713431 -> C328344
- R24: value 1K -> 1k
- RP1, RP2, RP3, RP4, RP7: LCSC C700514 -> C1980
- SW3: LCSC (none) -> C40735
- U10, U4, U5, U6, U7, U8, U9: footprint Package_SO:TSSOP-48_6.1x12.5mm_P0.5mm -> x68000-ext:TSSOP-48_6.1x12.5mm_P0.5mm
- U11: footprint x68000-ext:WM8804GEDS&slash_RV -> x68000-ext:WM8804GEDS-RV
- U19, U20: now not fitted; now left out of the parts list
- X1: footprint Oscillator:Oscillator_SMD_Abracon_ASV-4Pin_7.0x5.1mm -> Oscillator:Oscillator_SMD_Abracon_ASE-4Pin_3.2x2.5mm_HandSoldering; LCSC (none) -> C5203547
Connections:
- net MMC_ACCESS is gone; now on an unnamed net: U23.5 (A4)
- net GND: now also U23.19 (~{G2}), U23.6 (A5), C37.2, C38.2, J14.2 (Pin_2), LED1.GND (VSS), LED2.GND (VSS), NT1.1, SP1.2, U24.7 (VSS); no longer R24.2, U16.10 (DEMP)
- net GNDA: now also U16.10 (DEMP), NT1.2
- net I2C_SCL: now also SW3.2, U24.12 (PC2/SCL); no longer SW3.1
- net I2C_SCL_PI: now also SW3.3; no longer SW3.4
- net I2C_SDA: now also SW3.1, U24.11 (PC1/SDA); no longer SW3.2
- net I2C_SDA_PI: now also SW3.4; no longer SW3.3
- net MMC_CS: now also U24.20 (PD3)
- net MMC_MISO: now also U23.15 (Y4); no longer U23.14 (Y5)
- net VCC: now also J13.1 (Pin_1), LED1.VDD, LED2.VDD; no longer D12.1 (K)
- net WM8804_INTn: now also U24.19 (PD2); no longer U14.JP2_33 (GPIO_126)
- net at J11.7 (DAT0), RP9.3 (P3): no longer U23.6 (A5)
- net at R24.1: now also SP1.1
- net at U23.1 (~{G1}): now also JP1.2 (C)
- net +3V3 renamed +3.3V
- net +3.3V: now also C37.1, C38.1, R32.1, U24.9 (VDD)
- new net: D12.1 (K), J13.2 (Pin_2)
- new net: JP10.2 (C), LED2.DI (DIN)
- new net: JP10.3 (B), LED1.DO (DOUT)
- new net ENABLE_MMC_n: JP1.1 (A), U24.4 (PD7)
- new net KEPLERX_STATUS_LED: LED1.DI (DIN), U24.3 (PD6)
- new net MMC_ACCESS_LED: JP10.1 (A), U24.2 (PD5)
- new net MMC_DET_n: J11.9 (DET_B), JP1.3 (B), R32.2, U24.1 (PD4)
- new net SPEAKER: R24.2, U24.10 (PC0)
- new net SWIO: J14.1 (Pin_1), U14.JP2_33 (GPIO_126), U24.18 (PD1/SWIO)
- now unconnected: RP8.1 (P1)
- no-connect marks 61 -> 72
Other:
- moved on the sheet: C1, C13, C19, C2, C20, C3, C31, C32, C33, C35, C36, C8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

Commit message: V3.0.0 (Fixed)
Parts:
- U12, U13: LCSC (none) -> C2675018
- U3: value INA3221 -> INA3221AIRGVR; LCSC (none) -> C181255
- U4, U5, U6, U7, U8, U9: value 74LVC16374 -> 74LVC16374A
Connections:
- net GND: now also J14.1 (Pin_1); no longer J14.2 (Pin_2)
- net SWIO: now also J14.2 (Pin_2); no longer J14.1 (Pin_1)
Other:
- moved on the sheet: J14
Changed lines of the file:
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@@
       (effects (font (size 1.27 1.27)))
     )
-    (property "Value" "74LVC16374" (at 142.24 405.13 0)
+    (property "Value" "74LVC16374A" (at 142.24 405.13 0)
       (effects (font (size 1.27 1.27)))
     )
@@
     )
   )
-  (symbol (lib_id "Connector:Conn_01x02_Pin") (at 689.61 254 270) (unit 1)
-    (in_bom no) (on_board yes) (dnp yes) (fields_autoplaced)
-    (property "Reference" "J14" (at 690.88 253.3649 90)
+  (symbol (lib_id "Connector:Conn_01x02_Pin") (at 687.07 254 90) (mirror x) (unit 1)
+    (in_bom no) (on_board yes) (dnp yes)
+    (property "Reference" "J14" (at 685.8 253.3649 90)
       (effects (font (size 1.27 1.27)) (justify left))
     )
-    (property "Value" "Conn_01x02_Pin" (at 690.88 255.9049 90)
+    (property "Value" "Conn_01x02_Pin" (at 685.8 255.9049 90)
       (effects (font (size 1.27 1.27)) (justify left))
     )
-    (property "Footprint" "Connector_PinHeader_2.54mm:PinHeader_1x02_P2.54mm_Vertical" (at 689.61 254 0)
+    (property "Footprint" "Connector_PinHeader_2.54mm:PinHeader_1x02_P2.54mm_Vertical" (at 687.07 254 0)
       (effects (font (size 1.27 1.27)) hide)
     )
-    (property "Datasheet" "~" (at 689.61 254 0)
+    (property "Datasheet" "~" (at 687.07 254 0)
       (effects (font (size 1.27 1.27)) hide)
     )
@@
       (effects (font (size 1.27 1.27)))
     )
-    (property "Value" "74LVC16374" (at 142.24 101.6 0)
+    (property "Value" "74LVC16374A" (at 142.24 101.6 0)
       (effects (font (size 1.27 1.27)))
     )
@@
       (effects (font (size 1.27 1.27)))
     )
-    (property "Value" "74LVC16374" (at 142.24 175.26 0)
+    (property "Value" "74LVC16374A" (at 142.24 175.26 0)
       (effects (font (size 1.27 1.27)))
     )
@@
       (effects (font (size 1.27 1.27)) hide)
     )
-    (property "Datasheet" "" (at 234.95 527.05 0)
+    (property "Datasheet" "https://jlcpcb.com/partdetail/Toshiba-TC7MPB9307FT_EL/C2675018" (at 234.95 527.05 0)
+      (effects (font (size 1.27 1.27)) hide)
+    )
+    (property "LCSC" "C2675018" (at 234.95 527.05 0)
       (effects (font (size 1.27 1.27)) hide)
     )
@@
       (effects (font (size 1.27 1.27)) (justify left))
     )
-    (property "Value" "INA3221" (at 68.0594 155.575 0)
+    (property "Value" "INA3221AIRGVR" (at 68.0594 155.575 0)
       (effects (font (size 1.27 1.27)) (justify left))
     )
@@
       (effects (font (size 1.27 1.27)) hide)
     )
+    (property "LCSC" "C181255" (at 66.04 166.37 0)
+      (effects (font (size 1.27 1.27)) hide)
+    )
     (pin "1")
     (pin "10")
@@
       (effects (font (size 1.27 1.27)))
     )
-    (property "Value" "74LVC16374" (at 142.24 27.94 0)
+    (property "Value" "74LVC16374A" (at 142.24 27.94 0)
       (effects (font (size 1.27 1.27)))
     )
@@
       (effects (font (size 1.27 1.27)))
     )
-    (property "Value" "74LVC16374" (at 142.24 251.46 0)
+    (property "Value" "74LVC16374A" (at 142.24 251.46 0)
       (effects (font (size 1.27 1.27)))
     )
@@
       (effects (font (size 1.27 1.27)))
     )
-    (property "Value" "74LVC16374" (at 142.24 327.66 0)
+    (property "Value" "74LVC16374A" (at 142.24 327.66 0)
       (effects (font (size 1.27 1.27)))
     )
@@
       (effects (font (size 1.27 1.27)) hide)
     )
-    (property "Datasheet" "" (at 234.95 384.81 0)
+    (property "Datasheet" "https://jlcpcb.com/partdetail/Toshiba-TC7MPB9307FT_EL/C2675018" (at 234.95 384.81 0)
+      (effects (font (size 1.27 1.27)) hide)
+    )
+    (property "LCSC" "C2675018" (at 234.95 384.81 0)
       (effects (font (size 1.27 1.27)) hide)
     )
